File: UFO-FPGA/BANK1.kicad_sch (KiCad schematic)
At the start: 7 parts, among them U1 ICE40HX8K-BG121

Commit message: Added net labels
Connections:
- net VCCIO_1: now reaches C17.1, C17.1, C17.1, C18.1, R25.2, TP8.1, U1.F8 (VCCIO_1)
- net GND: now reaches C17.2, C17.2, C17.2, C18.2
Changed lines of the file:
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@@
   (junction (at 156.21 38.1) (diameter 0) (color 0 0 0 0)
   )
+  (junction (at 167.64 45.72) (diameter 0) (color 0 0 0 0)
+  )
   (junction (at 167.64 38.1) (diameter 0) (color 0 0 0 0)
   )
@@
   (wire (pts (xy 144.78 45.72) (xy 133.35 45.72))
     (stroke (width 0) (type default))
+  )
+  (label "VCCIO_1" (at 123.19 38.1 0) (fields_autoplaced)
+    (effects (font (size 1.27 1.27)) (justify left bottom))
   )
   (symbol (lib_id "FPGA_Lattice:ICE40HX8K-BG121") (at 123.19 82.55 0) (unit 2)
@@
         )
       )
+    )
+  )
+  (symbol (lib_id "power:GND") (at 167.64 45.72 0) (unit 1)
+    (in_bom yes) (on_board yes) (dnp no) (fields_autoplaced)
+    (property "Reference" "#PWR038" (at 167.64 52.07 0)
+      (effects (font (size 1.27 1.27)) hide)
+    )
+    (property "Value" "GND" (at 167.64 49.8555 0)
+      (effects (font (size 1.27 1.27)))
+    )
+    (property "Footprint" "" (at 167.64 45.72 0)
+      (effects (font (size 1.27 1.27)) hide)
+    )
+    (property "Datasheet" "" (at 167.64 45.72 0)
+      (effects (font (size 1.27 1.27)) hide)
+    )
+    (pin "1")
+    (instances
+      (project "UFO-FPGA"
+        (path "/b3168f6a-c732-41d3-aeeb-d97dd2f1bb65/f54d4357-d916-4d6b-afb9-9dd5f65d1cf7"
+          (reference "#PWR038") (unit 1)
+        )
+      )
