File: UFO-FPGA/UFO-FPGA.kicad_pcb (KiCad board)
At the start: 6 copper layers, 68.6 x 53.3 mm, 166 parts, among them J1 Power, J2 Digital, J3 Digital/PWM, J4 Digital, J5 USB_B_Micro, Q1 2N7002, SW1 SW_Push_DPDT, SW2 SW_DIP_x01, U1 ICE40HX8K-BG121, U11 TL071, U12 MAX11116AUT+T, U2 FT2232HL, U3 ASDMB-12MHz, U4 MC34063AD, U5 93LC56CT-I/MS, U6 PWR convert, U7 PWR convert, U9 N25Q032A13ESC40F

Commit message: PCB
Parts:
- removed PWR: POWER, LED_SMD:LED_0805_2012Metric_Pad1.15x1.40mm_HandSolder
- removed TP3: TestPoint, TestPoint:TestPoint_Keystone_5000-5004_Miniature
- added POWER1: POWER, LED_SMD:LED_0805_2012Metric_Pad1.15x1.40mm_HandSolder, F.Cu at (113.2, 96.0)
- C15, C16, C17, C18, C19, C20, D1, R25, R26: moved to B.Cu
- J2: footprint Connector_PinSocket_2.54mm:PinSocket_1x10_P2.54mm_Vertical -> Connector_PinSocket_2.54mm:PinSocket_1x06_P2.54mm_Vertical
- J3: footprint Connector_PinSocket_2.54mm:PinSocket_1x06_P2.54mm_Vertical -> Connector_PinSocket_2.54mm:PinSocket_1x10_P2.54mm_Vertical
- TP1, TP10, TP11, TP12, TP13, TP2, TP4, TP7, TP8, TP9: footprint TestPoint:TestPoint_Keystone_5000-5004_Miniature -> TestPoint:TestPoint_Pad_1.5x1.5mm
- TP5, TP6: footprint TestPoint:TestPoint_Keystone_5000-5004_Miniature -> TestPoint:TestPoint_Pad_1.5x1.5mm; moved to B.Cu
- moved U12 145.5 mm to (174.2, 61.5), turned to 180 degrees
- moved C58 142.6 mm to (170.8, 55.2)
- moved C57 142.4 mm to (170.8, 57.2), turned to 180 degrees
- moved R54 141.6 mm to (174.2, 57.2), turned to 180 degrees
- moved U11 131.0 mm to (165.8, 55.8), turned to 90 degrees
- moved C30 130.1 mm to (171.2, 73.2), turned to -90 degrees
- moved C29 127.9 mm to (168.3, 76.0)
- moved C31 126.4 mm to (168.2, 68.8)
- moved C32 126.4 mm to (168.2, 70.8)
- moved TP10 122.2 mm to (168.0, 73.2), turned to -90 degrees
- moved R31 122.0 mm to (168.2, 66.8), turned to 180 degrees
- moved SW1 121.6 mm to (178.8, 83.2), turned to -90 degrees
- moved C19 120.8 mm to (168.6, 76.0)
- moved TP4 120.6 mm to (170.2, 88.5), turned to 180 degrees
- moved SW2 119.6 mm to (177.2, 75.0), turned to 90 degrees
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Connections:
- net /BANK 4 - SPI Programming/2V5 renamed +2V5
- net /USB Programmer/FLASH-MISO renamed /USB Programmer/FLASH_MISO
- net /USB Programmer/FLASH-MOSI renamed /USB Programmer/FLASH_MOSI
- net Net-(C57-Pad2) renamed /ADC/Out-tl71
- net Net-(D6-K) renamed /Invert-5V-Dual-Ramp/-5Vled
- net Net-(U11-+) renamed /ADC/In-tl71
- J2 pad 5: AIN1 -> GND
- J2 pad 6: AIN2 -> AIN1_O
- R29 pad 1: +1V2 -> +3V3
- R30 pad 1: +1V2 -> +3V3
- R31 pad 1: +1V2 -> +3V3
- R32 pad 1: +1V2 -> +3V3
- U1 pad A1: PIN-1 -> unconnected-(U1A-IOT_225-PadA1)
- U1 pad A2: PIN-3 -> unconnected-(U1A-IOT_222-PadA2)
- U1 pad A3: PIN-2 -> unconnected-(U1A-IOT_223-PadA3)
- U1 pad A4: MISO -> unconnected-(U1A-IOT_211-PadA4)
- U1 pad A5: ADC-CS -> unconnected-(U1A-IOT_207-PadA5)
- U1 pad A6: SCK -> unconnected-(U1A-IOT_206-PadA6)
- U1 pad B1: PIN-9 -> unconnected-(U1D-IOL_2A-PadB1)
- U1 pad B11: PIN-23 -> unconnected-(U1B-IOR_161-PadB11)
- U1 pad B2: PIN-8 -> unconnected-(U1D-IOL_2B-PadB2)
- U1 pad B3: PIN-4 -> unconnected-(U1A-IOT_221-PadB3)
- U1 pad B4: PIN-5 -> unconnected-(U1A-IOT_219-PadB4)
- U1 pad B6: PIN-6 -> unconnected-(U1A-IOT_198_GBIN0-PadB6)
- U1 pad B7: PIN-7 -> unconnected-(U1A-IOT_197_GBIN1-PadB7)
- U1 pad C11: PIN-22 -> unconnected-(U1B-IOR_160-PadC11)
- U1 pad D11: PIN-21 -> unconnected-(U1B-IOR_152-PadD11)
- U1 pad E10: PIN-19 -> unconnected-(U1B-IOR_141_GBIN2-PadE10)
- U1 pad E11: PIN-20 -> unconnected-(U1B-IOR_148-PadE11)
- U1 pad F10: PIN-17 -> unconnected-(U1B-IOR_136-PadF10)
- U1 pad F11: PIN-18 -> unconnected-(U1B-IOR_140_GBIN3-PadF11)
- U1 pad G1: ICE_CLK -> unconnected-(U1D-IOL_14A_GBIN6-PadG1)
- U1 pad G10: PIN-15 -> unconnected-(U1B-IOR_120-PadG10)
- U1 pad G11: PIN-16 -> unconnected-(U1B-IOR_129-PadG11)
- U1 pad H10: PIN-12 -> unconnected-(U1B-IOR_116-PadH10)
- U1 pad H11: PIN-14 -> unconnected-(U1B-IOR_119-PadH11)
- U1 pad J10: PIN-13 -> unconnected-(U1B-IOR_117-PadJ10)
- U1 pad J11: PIN-10 -> unconnected-(U1B-IOR_114-PadJ11)
- U1 pad K1: RS232_Tx_TTL -> unconnected-(U1D-IOL_23B-PadK1)
- U1 pad K11: PIN-11 -> unconnected-(U1B-IOR_115-PadK11)
- U1 pad L1: RS232_Rx_TTL -> unconnected-(U1C-IOB_56-PadL1)
- U1 pad L2: RTSn -> unconnected-(U1C-IOB_61-PadL2)
- U1 pad L3: CTSn -> unconnected-(U1C-IOB_71-PadL3)
- U1 pad L4: DTRn -> unconnected-(U1C-IOB_72-PadL4)
- U1 pad L5: DSRn -> unconnected-(U1C-IOB_81_GBIN5-PadL5)
- U1 pad L7: DCDn -> unconnected-(U1C-IOB_94-PadL7)
