File: UFO-FPGA/untitled.kicad_sch (KiCad schematic)
At the start: 16 parts, among them U4 MC34063AD

Commit message: PCB planes
Added:
added Power plane +1v2, +3v3 and +5v on layer 4
Ground plane on layer 2 and 5
Added signal layer 1,3 and 6
Parts:
- C50, C54: footprint (none) -> Capacitor_SMD:CP_Elec_6.3x7.7
- C51: footprint (none) -> Capacitor_SMD:CP_Elec_8x10.5
- L1: footprint (none) -> Inductor_SMD:L_1210_3225Metric_Pad1.42x2.65mm_HandSolder
- L2: footprint (none) -> Inductor_SMD:L_1812_4532Metric_Pad1.30x3.40mm_HandSolder
Changed lines of the file:
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@@
       (effects (font (size 1.27 1.27)) (justify right))
     )
-    (property "Footprint" "" (at 133.0452 104.775 0)
+    (property "Footprint" "Capacitor_SMD:CP_Elec_8x10.5" (at 133.0452 104.775 0)
       (effects (font (size 1.27 1.27)) hide)
     )
@@
       (effects (font (size 1.27 1.27)) (justify right))
     )
-    (property "Footprint" "" (at 194.0052 104.775 0)
+    (property "Footprint" "Capacitor_SMD:CP_Elec_6.3x7.7" (at 194.0052 104.775 0)
       (effects (font (size 1.27 1.27)) hide)
     )
@@
       (effects (font (size 1.27 1.27)))
     )
-    (property "Footprint" "" (at 188.595 90.17 0)
+    (property "Footprint" "Inductor_SMD:L_1812_4532Metric_Pad1.30x3.40mm_HandSolder" (at 188.595 90.17 0)
       (effects (font (size 1.27 1.27)) hide)
     )
@@
       (effects (font (size 1.27 1.27)))
     )
-    (property "Footprint" "" (at 187.325 100.965 0)
+    (property "Footprint" "Inductor_SMD:L_1210_3225Metric_Pad1.42x2.65mm_HandSolder" (at 187.325 100.965 0)
       (effects (font (size 1.27 1.27)) hide)
     )
@@
       (effects (font (size 1.27 1.27)) (justify left))
     )
-    (property "Footprint" "" (at 115.2398 112.395 0)
-      (effects (font (size 1.27 1.27)) hide)
-    )
+    (property "Footprint" "Capacitor_SMD:CP_Elec_6.3x7.7" (at 115.2398 112.395 0)
+      (effects (font (size 1.27 1.27)) hide)
+    )

Commit message: PCB
Parts:
- TP13: footprint TestPoint:TestPoint_Keystone_5000-5004_Miniature -> TestPoint:TestPoint_Pad_1.5x1.5mm
Connections:
- net -5Vled: now reaches D6.1 (K), R48.2
Other:
- moved on the sheet: C49
Changed lines of the file:
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@@
   (junction (at 140.97 125.73) (diameter 0) (color 0 0 0 0)
   )
+  (junction (at 132.08 104.14) (diameter 0) (color 0 0 0 0)
+  )
   (junction (at 202.565 125.73) (diameter 0) (color 0 0 0 0)
   )
@@
   (junction (at 142.24 80.01) (diameter 0) (color 0 0 0 0)
   )
+  (junction (at 140.97 104.14) (diameter 0) (color 0 0 0 0)
+  )
   (junction (at 168.91 100.965) (diameter 0) (color 0 0 0 0)
   )
-  (junction (at 140.97 104.775) (diameter 0) (color 0 0 0 0)
-  )
   (junction (at 116.205 80.01) (diameter 0) (color 0 0 0 0)
   )
@@
   (junction (at 132.08 125.73) (diameter 0) (color 0 0 0 0)
   )
-  (junction (at 132.08 104.775) (diameter 0) (color 0 0 0 0)
-  )
   (junction (at 193.04 125.73) (diameter 0) (color 0 0 0 0)
   )
@@
     (stroke (width 0) (type default))
   )
+  (wire (pts (xy 120.65 98.425) (xy 120.65 99.06))
+    (stroke (width 0) (type default))
+  )
   (wire (pts (xy 142.24 80.01) (xy 142.24 82.55))
     (stroke (width 0) (type default))
@@
     (stroke (width 0) (type default))
   )
+  (wire (pts (xy 121.92 90.17) (xy 120.65 90.17))
+    (stroke (width 0) (type default))
+  )
   (wire (pts (xy 135.255 68.58) (xy 142.24 68.58))
     (stroke (width 0) (type default))
@@
     (stroke (width 0) (type default))
   )
-  (wire (pts (xy 132.08 104.775) (xy 140.97 104.775))
-    (stroke (width 0) (type default))
-  )
-  (wire (pts (xy 121.92 90.17) (xy 121.92 91.44))
+  (wire (pts (xy 132.08 104.14) (xy 140.97 104.14))
     (stroke (width 0) (type default))
   )
@@
     (stroke (width 0) (type default))
   )
+  (wire (pts (xy 120.65 90.17) (xy 120.65 90.805))
+    (stroke (width 0) (type default))
+  )
+  (wire (pts (xy 132.08 104.14) (xy 132.08 104.775))
+    (stroke (width 0) (type default))
+  )
   (wire (pts (xy 193.04 112.395) (xy 193.04 125.73))
     (stroke (width 0) (type default))
@@
     (stroke (width 0) (type default))
   )
-  (wire (pts (xy 132.08 99.06) (xy 132.08 104.775))
+  (wire (pts (xy 132.08 99.06) (xy 132.08 104.14))
     (stroke (width 0) (type default))
   )
@@
     (stroke (width 0) (type default))
   )
-  (wire (pts (xy 121.92 99.06) (xy 132.08 99.06))
+  (wire (pts (xy 120.65 99.06) (xy 132.08 99.06))
     (stroke (width 0) (type default))
   )
@@
     (fill (type none))
     (effects (font (size 1.27 1.27)) (justify left top))
+  )
+  (label "-5Vled" (at 202.565 114.935 0) (fields_autoplaced)
+    (effects (font (size 1.27 1.27)) (justify left bottom))
   )
   (label "-5 unfiltered" (at 168.91 104.14 0) (fields_autoplaced)
@@
     )
   )
+  (symbol (lib_id "power:PWR_FLAG") (at 202.565 100.965 270) (unit 1)
+    (in_bom yes) (on_board yes) (dnp no)
+    (property "Reference" "#FLG05" (at 204.47 100.965 0)
+      (effects (font (size 1.27 1.27)) hide)
+    )
+    (property "Value" "PWR_FLAG" (at 203.2 103.505 90)
+      (effects (font (size 1.27 1.27)) (justify left))
+    )
+    (property "Footprint" "" (at 202.565 100.965 0)
+      (effects (font (size 1.27 1.27)) hide)
+    )
+    (property "Datasheet" "~" (at 202.565 100.965 0)
+      (effects (font (size 1.27 1.27)) hide)
+    )
+    (pin "1")
+    (instances
+      (project "UFO-FPGA"
+        (path "/b3168f6a-c732-41d3-aeeb-d97dd2f1bb65/4b884ea1-5945-4826-a315-db89106495d4"
+          (reference "#FLG05") (unit 1)
+        )
+      )
+    )
+  )
   (symbol (lib_id "Device:C") (at 140.97 108.585 0) (unit 1)
     (in_bom yes) (on_board yes) (dnp no) (fields_autoplaced)
@@
       (effects (font (size 1.27 1.27)) (justify left))
     )
-    (property "Footprint" "TestPoint:TestPoint_Keystone_5000-5004_Miniature" (at 207.645 100.33 0)
+    (property "Footprint" "TestPoint:TestPoint_Pad_1.5x1.5mm" (at 207.645 100.33 0)
       (effects (font (size 1.27 1.27)) hide)
     )
@@
     )
   )
-  (symbol (lib_id "Device:C") (at 121.92 95.25 0) (unit 1)
-    (in_bom yes) (on_board yes) (dnp no) (fields_autoplaced)
-    (property "Reference" "C49" (at 124.841 94.6063 0)
-      (effects (font (size 1.27 1.27)) (justify left))
-    )
-    (property "Value" "220pF" (at 124.841 96.5273 0)
-      (effects (font (size 1.27 1.27)) (justify left))
-    )
-    (property "Footprint" "Capacitor_SMD:C_0805_2012Metric_Pad1.18x1.45mm_HandSolder" (at 122.8852 99.06 0)
-      (effects (font (size 1.27 1.27)) hide)
-    )
-    (property "Datasheet" "~" (at 121.92 95.25 0)
-      (effects (font (size 1.27 1.27)) hide)
-    )
+  (symbol (lib_id "Device:C") (at 120.65 94.615 0) (mirror y) (unit 1)
+    (in_bom yes) (on_board yes) (dnp no)
+    (property "Reference" "C49" (at 117.729 93.9713 0)
+      (effects (font (size 1.27 1.27)) (justify left))
+    )
+    (property "Value" "220pF" (at 117.729 95.8923 0)
+      (effects (font (size 1.27 1.27)) (justify left))
+    )
+    (property "Footprint" "Capacitor_SMD:C_0805_2012Metric_Pad1.18x1.45mm_HandSolder" (at 119.6848 98.425 0)
+      (effects (font (size 1.27 1.27)) hide)
+    )
+    (property "Datasheet" "~" (at 120.65 94.615 0)
+      (effects (font (size 1.27 1.27)) hide)
+    )
