File: UFO-FPGA/POWER.kicad_sch (KiCad schematic)
At the start: 42 parts, among them J5 USB_B_Micro, Q1 2N7002, U6 PWR convert, U7 PWR convert

Commit message: footprints and PCB
Parts:
- D5: value LED -> POWER; footprint (none) -> LED_SMD:LED_0805_2012Metric_Pad1.15x1.40mm_HandSolder
- FB1: footprint (none) -> Inductor_SMD:L_1206_3216Metric_Pad1.22x1.90mm_HandSolder
- R35, R36, R37, R45, R47, R48: footprint (none) -> Resistor_SMD:R_0805_2012Metric_Pad1.20x1.40mm_HandSolder
- R46: value R -> 1K; footprint (none) -> Resistor_SMD:R_0805_2012Metric_Pad1.20x1.40mm_HandSolder
- TP1: footprint (none) -> TestPoint:TestPoint_Keystone_5000-5004_Miniature
Changed lines of the file:
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@@
       (effects (font (size 1.27 1.27)) (justify right))
     )
-    (property "Footprint" "" (at 134.493 99.06 90)
+    (property "Footprint" "Resistor_SMD:R_0805_2012Metric_Pad1.20x1.40mm_HandSolder" (at 134.493 99.06 90)
       (effects (font (size 1.27 1.27)) hide)
     )
@@
       (effects (font (size 1.27 1.27)) (justify right))
     )
-    (property "Footprint" "" (at 94.488 43.815 90)
+    (property "Footprint" "Resistor_SMD:R_0805_2012Metric_Pad1.20x1.40mm_HandSolder" (at 94.488 43.815 90)
       (effects (font (size 1.27 1.27)) hide)
     )
@@
       (effects (font (size 1.27 1.27)) (justify right))
     )
-    (property "Footprint" "" (at 229.87 91.44 0)
+    (property "Footprint" "TestPoint:TestPoint_Keystone_5000-5004_Miniature" (at 229.87 91.44 0)
       (effects (font (size 1.27 1.27)) hide)
     )
@@
       (effects (font (size 1.27 1.27)) (justify right))
     )
-    (property "Footprint" "" (at 252.73 91.44 0)
+    (property "Footprint" "TestPoint:TestPoint_Keystone_5000-5004_Miniature" (at 252.73 91.44 0)
       (effects (font (size 1.27 1.27)) hide)
     )
@@
       (effects (font (size 1.27 1.27)) (justify left))
     )
-    (property "Footprint" "" (at 43.307 93.98 90)
+    (property "Footprint" "Inductor_SMD:L_1206_3216Metric_Pad1.22x1.90mm_HandSolder" (at 43.307 93.98 90)
       (effects (font (size 1.27 1.27)) hide)
     )
@@
       (effects (font (size 1.27 1.27)) (justify right))
     )
-    (property "Footprint" "" (at 241.3 91.44 0)
+    (property "Footprint" "TestPoint:TestPoint_Keystone_5000-5004_Miniature" (at 241.3 91.44 0)
       (effects (font (size 1.27 1.27)) hide)
     )
@@
       (effects (font (size 1.27 1.27)) (justify right))
     )
-    (property "Footprint" "" (at 119.253 102.87 90)
+    (property "Footprint" "Resistor_SMD:R_0805_2012Metric_Pad1.20x1.40mm_HandSolder" (at 119.253 102.87 90)
       (effects (font (size 1.27 1.27)) hide)
     )
@@
       (effects (font (size 1.27 1.27)))
     )
-    (property "Value" "R" (at 80.01 86.7951 90)
-      (effects (font (size 1.27 1.27)))
-    )
-    (property "Footprint" "" (at 80.01 90.678 90)
+    (property "Value" "1K" (at 80.01 86.7951 90)
+      (effects (font (size 1.27 1.27)))
+    )
+    (property "Footprint" "Resistor_SMD:R_0805_2012Metric_Pad1.20x1.40mm_HandSolder" (at 80.01 90.678 90)
       (effects (font (size 1.27 1.27)) hide)
     )
@@
       (effects (font (size 1.27 1.27)) (justify right))
     )
-    (property "Footprint" "" (at 219.71 91.44 0)
+    (property "Footprint" "TestPoint:TestPoint_Keystone_5000-5004_Miniature" (at 219.71 91.44 0)
       (effects (font (size 1.27 1.27)) hide)
     )
@@
       (effects (font (size 1.27 1.27)) (justify right))
     )
-    (property "Value" "LED" (at 89.281 98.7498 90)
-      (effects (font (size 1.27 1.27)) (justify right))
-    )
-    (property "Footprint" "" (at 86.36 95.885 0)
+    (property "Value" "POWER" (at 89.281 98.7498 90)
+      (effects (font (size 1.27 1.27)) (justify right))
+    )
+    (property "Footprint" "LED_SMD:LED_0805_2012Metric_Pad1.15x1.40mm_HandSolder" (at 86.36 95.885 0)
       (effects (font (size 1.27 1.27)) hide)
     )
@@
       (effects (font (size 1.27 1.27)) (justify right))
     )
-    (property "Footprint" "" (at 40.132 35.56 90)
+    (property "Footprint" "Resistor_SMD:R_0805_2012Metric_Pad1.20x1.40mm_HandSolder" (at 40.132 35.56 90)
       (effects (font (size 1.27 1.27)) hide)
     )
@@
       (effects (font (size 1.27 1.27)))
     )
-    (property "Footprint" "" (at 102.235 25.273 90)
+    (property "Footprint" "Resistor_SMD:R_0805_2012Metric_Pad1.20x1.40mm_HandSolder" (at 102.235 25.273 90)
       (effects (font (size 1.27 1.27)) hide)
     )
@@
       (effects (font (size 1.27 1.27)) (justify right))
     )
-    (property "Footprint" "" (at 94.488 32.385 90)
+    (property "Footprint" "Resistor_SMD:R_0805_2012Metric_Pad1.20x1.40mm_HandSolder" (at 94.488 32.385 90)
       (effects (font (size 1.27 1.27)) hide)
     )
@@
       (effects (font (size 1.27 1.27)))
     )
-    (property "Footprint" "" (at 65.405 114.808 90)
-      (effects (font (size 1.27 1.27)) hide)
-    )
+    (property "Footprint" "Resistor_SMD:R_0805_2012Metric_Pad1.20x1.40mm_HandSolder" (at 65.405 114.808 90)
+      (effects (font (size 1.27 1.27)) hide)
+    )

Commit message: footprint
Parts:
- C14, C2, C3, C38, C39, C4, C42, C43, C49, C5, C50, C6: footprint (none) -> Capacitor_SMD:C_0805_2012Metric_Pad1.18x1.45mm_HandSolder
- R38, R39, R40: footprint (none) -> Resistor_SMD:R_0805_2012Metric
Changed lines of the file:
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@@
       (effects (font (size 1.27 1.27)))
     )
-    (property "Footprint" "" (at 69.215 118.4402 0)
+    (property "Footprint" "Capacitor_SMD:C_0805_2012Metric_Pad1.18x1.45mm_HandSolder" (at 69.215 118.4402 0)
       (effects (font (size 1.27 1.27)) hide)
     )
@@
       (effects (font (size 1.27 1.27)))
     )
-    (property "Footprint" "" (at 234.95 25.908 90)
+    (property "Footprint" "Resistor_SMD:R_0805_2012Metric" (at 234.95 25.908 90)
       (effects (font (size 1.27 1.27)) hide)
     )
@@
       (effects (font (size 1.27 1.27)) (justify left))
     )
-    (property "Footprint" "" (at 188.9252 97.155 0)
+    (property "Footprint" "Capacitor_SMD:C_0805_2012Metric_Pad1.18x1.45mm_HandSolder" (at 188.9252 97.155 0)
       (effects (font (size 1.27 1.27)) hide)
     )
@@
       (effects (font (size 1.27 1.27)) (justify left))
     )
-    (property "Footprint" "" (at 234.6452 36.83 0)
+    (property "Footprint" "Capacitor_SMD:C_0805_2012Metric_Pad1.18x1.45mm_HandSolder" (at 234.6452 36.83 0)
       (effects (font (size 1.27 1.27)) hide)
     )
@@
       (effects (font (size 1.27 1.27)) (justify left))
     )
-    (property "Footprint" "" (at 53.0352 55.88 0)
+    (property "Footprint" "Capacitor_SMD:C_0805_2012Metric_Pad1.18x1.45mm_HandSolder" (at 53.0352 55.88 0)
       (effects (font (size 1.27 1.27)) hide)
     )
@@
       (effects (font (size 1.27 1.27)) (justify left))
     )
-    (property "Footprint" "" (at 152.7302 97.155 0)
+    (property "Footprint" "Capacitor_SMD:C_0805_2012Metric_Pad1.18x1.45mm_HandSolder" (at 152.7302 97.155 0)
       (effects (font (size 1.27 1.27)) hide)
     )
@@
       (effects (font (size 1.27 1.27)) (justify left))
     )
-    (property "Footprint" "" (at 181.9402 117.475 0)
+    (property "Footprint" "Capacitor_SMD:C_0805_2012Metric_Pad1.18x1.45mm_HandSolder" (at 181.9402 117.475 0)
       (effects (font (size 1.27 1.27)) hide)
     )
@@
       (effects (font (size 1.27 1.27)) (justify left))
     )
-    (property "Footprint" "" (at 154.0002 117.475 0)
+    (property "Footprint" "Capacitor_SMD:C_0805_2012Metric_Pad1.18x1.45mm_HandSolder" (at 154.0002 117.475 0)
       (effects (font (size 1.27 1.27)) hide)
     )
@@
       (effects (font (size 1.27 1.27)))
     )
-    (property "Footprint" "" (at 74.5998 100.33 0)
+    (property "Footprint" "Capacitor_SMD:C_0805_2012Metric_Pad1.18x1.45mm_HandSolder" (at 74.5998 100.33 0)
       (effects (font (size 1.27 1.27)) hide)
     )
@@
       (effects (font (size 1.27 1.27)) (justify left))
     )
-    (property "Footprint" "" (at 105.7402 36.195 0)
+    (property "Footprint" "Capacitor_SMD:C_0805_2012Metric_Pad1.18x1.45mm_HandSolder" (at 105.7402 36.195 0)
       (effects (font (size 1.27 1.27)) hide)
     )
@@
       (effects (font (size 1.27 1.27)) (justify right))
     )
-    (property "Footprint" "" (at 227.203 44.45 90)
+    (property "Footprint" "Resistor_SMD:R_0805_2012Metric" (at 227.203 44.45 90)
       (effects (font (size 1.27 1.27)) hide)
     )
@@
       (effects (font (size 1.27 1.27)) (justify left))
     )
-    (property "Footprint" "" (at 170.5102 97.155 0)
+    (property "Footprint" "Capacitor_SMD:C_0805_2012Metric_Pad1.18x1.45mm_HandSolder" (at 170.5102 97.155 0)
       (effects (font (size 1.27 1.27)) hide)
     )
@@
       (effects (font (size 1.27 1.27)) (justify left))
     )
-    (property "Footprint" "" (at 198.4502 97.155 0)
+    (property "Footprint" "Capacitor_SMD:C_0805_2012Metric_Pad1.18x1.45mm_HandSolder" (at 198.4502 97.155 0)
       (effects (font (size 1.27 1.27)) hide)
     )
@@
       (effects (font (size 1.27 1.27)) (justify left))
     )
-    (property "Footprint" "" (at 207.9752 97.155 0)
+    (property "Footprint" "Capacitor_SMD:C_0805_2012Metric_Pad1.18x1.45mm_HandSolder" (at 207.9752 97.155 0)
       (effects (font (size 1.27 1.27)) hide)
     )
@@
       (effects (font (size 1.27 1.27)) (justify left))
     )
-    (property "Footprint" "" (at 172.4152 117.475 0)
+    (property "Footprint" "Capacitor_SMD:C_0805_2012Metric_Pad1.18x1.45mm_HandSolder" (at 172.4152 117.475 0)
       (effects (font (size 1.27 1.27)) hide)
     )
@@
       (effects (font (size 1.27 1.27)) (justify left))
     )
-    (property "Footprint" "" (at 180.0352 97.155 0)
+    (property "Footprint" "Capacitor_SMD:C_0805_2012Metric_Pad1.18x1.45mm_HandSolder" (at 180.0352 97.155 0)
       (effects (font (size 1.27 1.27)) hide)
     )
@@
       (effects (font (size 1.27 1.27)) (justify right))
     )
-    (property "Footprint" "" (at 227.203 33.02 90)
+    (property "Footprint" "Resistor_SMD:R_0805_2012Metric" (at 227.203 33.02 90)
       (effects (font (size 1.27 1.27)) hide)
     )
@@
       (effects (font (size 1.27 1.27)) (justify left))
     )
-    (property "Footprint" "" (at 161.6202 97.155 0)
+    (property "Footprint" "Capacitor_SMD:C_0805_2012Metric_Pad1.18x1.45mm_HandSolder" (at 161.6202 97.155 0)
       (effects (font (size 1.27 1.27)) hide)
     )
@@
       (effects (font (size 1.27 1.27)) (justify left))
     )
-    (property "Footprint" "" (at 185.7502 56.515 0)
+    (property "Footprint" "Capacitor_SMD:C_0805_2012Metric_Pad1.18x1.45mm_HandSolder" (at 185.7502 56.515 0)
       (effects (font (size 1.27 1.27)) hide)
     )
@@
       (effects (font (size 1.27 1.27)) (justify left))
     )
-    (property "Footprint" "" (at 162.8902 117.475 0)
-      (effects (font (size 1.27 1.27)) hide)
-    )
+    (property "Footprint" "Capacitor_SMD:C_0805_2012Metric_Pad1.18x1.45mm_HandSolder" (at 162.8902 117.475 0)
+      (effects (font (size 1.27 1.27)) hide)
+    )

Commit message: Footprints and values
Parts:
- added R36: 400, Resistor_SMD:R_0805_2012Metric_Pad1.20x1.40mm_HandSolder, symbol Device:R
- added R37: 900, Resistor_SMD:R_0805_2012Metric_Pad1.20x1.40mm_HandSolder, symbol Device:R
- added R39: 750R, Resistor_SMD:R_0805_2012Metric, symbol Device:R
- R36: value 12K4 -> 12k
- R37: value 24K9 -> 24k
- R38: value 11.8k -> 12k
- R39: value 3.74k -> 3k
Connections:
- net GND: now also R37.1, R39.1; no longer R37.1, R39.1
- net at C38.2, R37.2, U6.3 (FB): now also R36.1; no longer R36.1
- new net: R37.1, R37.2
- new net: R39.1, R39.2
- new net: R36.1, R36.2
Other:
- moved on the sheet: R36, R37

Commit message: PCB planes
Added:
added Power plane +1v2, +3v3 and +5v on layer 4
Ground plane on layer 2 and 5
Added signal layer 1,3 and 6
Parts:
- C37, C40, C41, C44: footprint (none) -> Capacitor_SMD:C_1206_3216Metric_Pad1.33x1.80mm_HandSolder
Changed lines of the file:
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@@
       (effects (font (size 1.27 1.27)) (justify left))
     )
-    (property "Footprint" "" (at 122.2502 36.195 0)
+    (property "Footprint" "Capacitor_SMD:C_1206_3216Metric_Pad1.33x1.80mm_HandSolder" (at 122.2502 36.195 0)
       (effects (font (size 1.27 1.27)) hide)
     )
@@
       (effects (font (size 1.27 1.27)) (justify left))
     )
-    (property "Footprint" "" (at 46.0248 33.655 0)
+    (property "Footprint" "Capacitor_SMD:C_1206_3216Metric_Pad1.33x1.80mm_HandSolder" (at 46.0248 33.655 0)
       (effects (font (size 1.27 1.27)) hide)
     )
@@
       (effects (font (size 1.27 1.27)) (justify left))
     )
-    (property "Footprint" "" (at 243.5352 36.83 0)
+    (property "Footprint" "Capacitor_SMD:C_1206_3216Metric_Pad1.33x1.80mm_HandSolder" (at 243.5352 36.83 0)
       (effects (font (size 1.27 1.27)) hide)
     )
@@
       (effects (font (size 1.27 1.27)) (justify left))
     )
-    (property "Footprint" "" (at 183.8198 34.29 0)
+    (property "Footprint" "Capacitor_SMD:C_1206_3216Metric_Pad1.33x1.80mm_HandSolder" (at 183.8198 34.29 0)
       (effects (font (size 1.27 1.27)) hide)
     )
@@
       (project "UFO-FPGA"
         (path "/b3168f6a-c732-41d3-aeeb-d97dd2f1bb65/abe08156-b909-4d2d-ad35-f723f4a728d5"
-          (reference "D7") (unit 1)
-        )
-      )
+          (reference "POWER1") (unit 1)
+        )
+      )

Commit message: ubs shield
Connections:
- no-connect marks 14 -> 15
Changed lines of the file:
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@@
   (no_connect (at 86.995 40.64))
   (no_connect (at 219.71 53.975))
+  (no_connect (at 32.385 118.11))
   (no_connect (at 86.995 45.72))
   (no_connect (at 86.995 43.18))

Commit message: PCB
Parts:
- removed TP1: TestPoint, TestPoint:TestPoint_Keystone_5000-5004_Miniature, symbol Connector:TestPoint
- TP1: footprint TestPoint:TestPoint_Keystone_5000-5004_Miniature -> TestPoint:TestPoint_Pad_1.5x1.5mm

Commit message: PCB
many pcb changes
-started routing
-added vias
-power planes
-ground planes
Parts:
- removed C14, C5: 100nF, Capacitor_SMD:C_0805_2012Metric_Pad1.18x1.45mm_HandSolder, symbol Device:C
- removed R36: 400, Resistor_SMD:R_0805_2012Metric_Pad1.20x1.40mm_HandSolder, symbol Device:R
- removed R36: 12k, Resistor_SMD:R_0805_2012Metric_Pad1.20x1.40mm_HandSolder, symbol Device:R
- removed R37: 24k, Resistor_SMD:R_0805_2012Metric_Pad1.20x1.40mm_HandSolder, symbol Device:R
- removed R37: 900, Resistor_SMD:R_0805_2012Metric_Pad1.20x1.40mm_HandSolder, symbol Device:R
- removed R38: 12k, Resistor_SMD:R_0805_2012Metric, symbol Device:R
- removed R39: 750R, Resistor_SMD:R_0805_2012Metric, symbol Device:R
- removed R39: 3k, Resistor_SMD:R_0805_2012Metric, symbol Device:R
- C4, C6: value 100nF -> 200nF
Connections:
- net +1V2: now also U6.2 (SNS)
- net +3V3: now also U7.2 (SNS)
- net GND: now also U6.9 (400mV), U7.10 (800mV), U7.11 (1.6V), U7.6 (100mV)
- net +3V3FB: now reaches C43.2, U7.3 (FB)
- net +1v2NR/ss: now reaches C39.1, U6.13 (NR/SS)
- net +1v2FB: now reaches C38.2, U6.3 (FB)
- net +3v3NR/ss: now reaches C42.1, U7.13 (NR/SS)
- net +1v2en: now reaches R48.1, U6.14 (EN)
- no-connect marks 15 -> 10
Other:
- moved on the sheet: C14, C6

Commit message: pcb prog redesign
Parts:
- J5: footprint Connector_USB:USB_Micro-AB_Molex_47590-0001 -> Connector_USB:USB_Micro-B_GCT_USB3076-30-A
Connections:
- net DM renamed D-
- net DP renamed D+
Changed lines of the file:
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@@
     (effects (font (size 1.27 1.27)) (justify left bottom))
   )
-  (global_label "DP" (shape input) (at 49.53 107.95 0) (fields_autoplaced)
+  (global_label "D+" (shape input) (at 49.53 107.95 0) (fields_autoplaced)
     (effects (font (size 1.27 1.27)) (justify left))
-    (property "Intersheetrefs" "${INTERSHEET_REFS}" (at 54.9758 107.95 0)
+    (property "Intersheetrefs" "${INTERSHEET_REFS}" (at 55.2782 107.95 0)
       (effects (font (size 1.27 1.27)) (justify left) hide)
     )
@@
     )
   )
-  (global_label "DM" (shape input) (at 49.53 110.49 0) (fields_autoplaced)
+  (global_label "D-" (shape input) (at 49.53 110.49 0) (fields_autoplaced)
     (effects (font (size 1.27 1.27)) (justify left))
-    (property "Intersheetrefs" "${INTERSHEET_REFS}" (at 55.1572 110.49 0)
+    (property "Intersheetrefs" "${INTERSHEET_REFS}" (at 55.2782 110.49 0)
       (effects (font (size 1.27 1.27)) (justify left) hide)
     )
@@
       (effects (font (size 1.27 1.27)))
     )
-    (property "Footprint" "Connector_USB:USB_Micro-AB_Molex_47590-0001" (at 38.735 109.22 0)
-      (effects (font (size 1.27 1.27)) hide)
-    )
+    (property "Footprint" "Connector_USB:USB_Micro-B_GCT_USB3076-30-A" (at 38.735 109.22 0)
+      (effects (font (size 1.27 1.27)) hide)
+    )
