File: UFO-FPGA/PINOUT.kicad_sch (KiCad schematic)
At the start: 4 parts, among them J1 Power, J2 Digital, J3 Digital/PWM, J4 Digital

Commit message: pcb
added monkey
Connections:
- net GND: no longer J1.8 (Pin_8), J2.5 (Pin_5)
- net PIN-18: now also J2.5 (Pin_5); no longer J2.1 (Pin_1)
- net PIN-19: now also J2.4 (Pin_4); no longer J2.2 (Pin_2)
- net PIN-21: now also J2.2 (Pin_2); no longer J2.4 (Pin_4)
- net PIN-22: now also J2.1 (Pin_1); no longer J1.1 (Pin_1)
- net PIN-23: now also J1.3 (Pin_3); no longer J1.2 (Pin_2)
- net PIN-24: now also J1.2 (Pin_2); no longer J1.3 (Pin_3)
- new net PIN-25: J1.1 (Pin_1)
- no-connect marks 0 -> 1
