File: UFO-FPGA/BANK4.kicad_sch (KiCad schematic)
At the start: 20 parts, among them SW1 SW_Push_DPDT, SW2 SW_DIP_x01, U1 ICE40HX8K-BG121, U9 N25Q032A13ESC40F

Commit message: PCB planes
Added:
added Power plane +1v2, +3v3 and +5v on layer 4
Ground plane on layer 2 and 5
Added signal layer 1,3 and 6
Parts:
- SW1: footprint (none) -> Button_Switch_THT:SW_CuK_JS202011CQN_DPDT_Straight
Changed lines of the file:
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@@
       (effects (font (size 1.27 1.27)))
     )
-    (property "Footprint" "" (at 72.39 158.75 0)
+    (property "Footprint" "Button_Switch_THT:SW_CuK_JS202011CQN_DPDT_Straight" (at 72.39 158.75 0)
       (effects (font (size 1.27 1.27)) hide)
     )

Commit message: PCB
Parts:
- TP1: footprint TestPoint:TestPoint_Keystone_5000-5004_Miniature -> TestPoint:TestPoint_Pad_1.5x1.5mm
Connections:
- net 2V5 renamed +2V5
Other:
- moved on the sheet: D1
Changed lines of the file:
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@@
   (junction (at 83.82 71.12) (diameter 0) (color 0 0 0 0)
+  )
+  (junction (at 109.22 48.895) (diameter 0) (color 0 0 0 0)
+  )
+  (junction (at 109.22 50.8) (diameter 0) (color 0 0 0 0)
   )
   (junction (at 73.66 71.12) (diameter 0) (color 0 0 0 0)
@@
     (stroke (width 0) (type default))
   )
-  (wire (pts (xy 109.22 44.45) (xy 109.22 40.64))
-    (stroke (width 0) (type default))
-  )
   (wire (pts (xy 162.56 40.64) (xy 205.74 40.64))
     (stroke (width 0) (type default))
@@
     (stroke (width 0) (type default))
   )
+  (wire (pts (xy 109.22 48.895) (xy 109.22 50.8))
+    (stroke (width 0) (type default))
+  )
   (wire (pts (xy 73.66 71.12) (xy 83.82 71.12))
     (stroke (width 0) (type default))
@@
     (stroke (width 0) (type default))
   )
-  (wire (pts (xy 109.22 52.07) (xy 109.22 53.34))
+  (wire (pts (xy 109.22 48.26) (xy 109.22 48.895))
     (stroke (width 0) (type default))
   )
@@
   )
   (wire (pts (xy 83.82 73.66) (xy 93.98 73.66))
+    (stroke (width 0) (type default))
+  )
+  (wire (pts (xy 109.22 50.8) (xy 109.22 53.34))
     (stroke (width 0) (type default))
   )
@@
   )
   (label "VCCPLL1" (at 73.66 73.66 0) (fields_autoplaced)
-    (effects (font (size 1.27 1.27)) (justify left bottom))
-  )
-  (label "2V5" (at 109.22 53.34 0) (fields_autoplaced)
     (effects (font (size 1.27 1.27)) (justify left bottom))
   )
@@
       (effects (font (size 1.27 1.27)) (justify left))
     )
-    (property "Footprint" "TestPoint:TestPoint_Keystone_5000-5004_Miniature" (at 63.5 63.5 0)
+    (property "Footprint" "TestPoint:TestPoint_Pad_1.5x1.5mm" (at 63.5 63.5 0)
       (effects (font (size 1.27 1.27)) hide)
     )
@@
       (effects (font (size 1.27 1.27)))
     )
-    (property "Footprint" "TestPoint:TestPoint_Keystone_5000-5004_Miniature" (at 52.07 77.47 0)
+    (property "Footprint" "TestPoint:TestPoint_Pad_1.5x1.5mm" (at 52.07 77.47 0)
       (effects (font (size 1.27 1.27)) hide)
     )
@@
         (path "/b3168f6a-c732-41d3-aeeb-d97dd2f1bb65/8a110dcf-7b5f-4510-96dd-3ef5ec8aca05"
           (reference "#PWR037") (unit 1)
+        )
+      )
+    )
+  )
+  (symbol (lib_id "power:PWR_FLAG") (at 109.22 50.8 270) (unit 1)
+    (in_bom yes) (on_board yes) (dnp no) (fields_autoplaced)
+    (property "Reference" "#FLG04" (at 111.125 50.8 0)
+      (effects (font (size 1.27 1.27)) hide)
+    )
+    (property "Value" "PWR_FLAG" (at 112.395 51.1168 90)
+      (effects (font (size 1.27 1.27)) (justify left))
+    )
+    (property "Footprint" "" (at 109.22 50.8 0)
+      (effects (font (size 1.27 1.27)) hide)
+    )
+    (property "Datasheet" "~" (at 109.22 50.8 0)
+      (effects (font (size 1.27 1.27)) hide)
+    )
+    (pin "1")
+    (instances
+      (project "UFO-FPGA"
+        (path "/b3168f6a-c732-41d3-aeeb-d97dd2f1bb65/a9a0295d-b075-4952-a5ba-04debc5f691c"
+          (reference "#FLG04") (unit 1)
         )
       )
@@
       (effects (font (size 1.27 1.27)) (justify right))
     )
-    (property "Footprint" "TestPoint:TestPoint_Keystone_5000-5004_Miniature" (at 68.58 77.47 0)
+    (property "Footprint" "TestPoint:TestPoint_Pad_1.5x1.5mm" (at 68.58 77.47 0)
       (effects (font (size 1.27 1.27)) hide)
     )
@@
     )
   )
-  (symbol (lib_id "Diode:CD4148W") (at 109.22 48.26 90) (unit 1)
+  (symbol (lib_id "Diode:CD4148W") (at 109.22 44.45 90) (unit 1)
     (in_bom yes) (on_board yes) (dnp no)
-    (property "Reference" "D1" (at 110.49 46.339 90)
+    (property "Reference" "D1" (at 110.49 42.529 90)
       (effects (font (size 1.27 1.27)) (justify right))
     )
-    (property "Value" "CDSU4148" (at 110.49 48.26 90)
+    (property "Value" "CDSU4148" (at 110.49 44.45 90)
       (effects (font (size 1.27 1.27)) (justify right))
     )
-    (property "Footprint" "Diode_SMD:D_0805_2012Metric_Pad1.15x1.40mm_HandSolder" (at 114.3 48.26 0)
-      (effects (font (size 1.27 1.27)) hide)
-    )
-    (property "Datasheet" "https://www.dccomponents.com/upload/product/original/623524775088.pdf" (at 109.22 48.26 0)
-      (effects (font (size 1.27 1.27)) hide)
-    )
-    (property "Sim.Device" "D" (at 109.22 48.26 0)
-      (effects (font (size 1.27 1.27)) hide)
-    )
-    (property "Sim.Pins" "1=K 2=A" (at 109.22 48.26 0)
+    (property "Footprint" "Diode_SMD:D_0805_2012Metric_Pad1.15x1.40mm_HandSolder" (at 114.3 44.45 0)
+      (effects (font (size 1.27 1.27)) hide)
+    )
+    (property "Datasheet" "https://www.dccomponents.com/upload/product/original/623524775088.pdf" (at 109.22 44.45 0)
+      (effects (font (size 1.27 1.27)) hide)
+    )
+    (property "Sim.Device" "D" (at 109.22 44.45 0)
+      (effects (font (size 1.27 1.27)) hide)
+    )
+    (property "Sim.Pins" "1=K 2=A" (at 109.22 44.45 0)
       (effects (font (size 1.27 1.27)) hide)
     )
@@
         )
       )
+    )
+  )
+  (symbol (lib_id "power:+2V5") (at 109.22 48.895 270) (unit 1)
+    (in_bom yes) (on_board yes) (dnp no)
+    (property "Reference" "#PWR061" (at 105.41 48.895 0)
+      (effects (font (size 1.27 1.27)) hide)
+    )
+    (property "Value" "+2V5" (at 109.855 46.99 90)
+      (effects (font (size 1.27 1.27)) (justify left))
+    )
+    (property "Footprint" "" (at 109.22 48.895 0)
+      (effects (font (size 1.27 1.27)) hide)
+    )
+    (property "Datasheet" "" (at 109.22 48.895 0)
+      (effects (font (size 1.27 1.27)) hide)
+    )
+    (pin "1")
+    (instances
+      (project "UFO-FPGA"
+        (path "/b3168f6a-c732-41d3-aeeb-d97dd2f1bb65/a9a0295d-b075-4952-a5ba-04debc5f691c"
+          (reference "#PWR061") (unit 1)
+        )
+      )

Commit message: pcb prog redesign
Parts:
- removed SW1: SW_Push_DPDT, Button_Switch_THT:SW_CuK_JS202011CQN_DPDT_Straight, symbol Switch:SW_Push_DPDT
- removed SW2: SW_DIP_x01, Button_Switch_SMD:SW_DIP_SPSTx01_Slide_9.78x4.72mm_W8.61mm_P2.54mm, symbol Switch:SW_DIP_x01
- added J6: Conn_02x02_Counter_Clockwise, Connector_PinHeader_2.54mm:PinHeader_2x02_P2.54mm_Vertical, symbol Connector_Generic:Conn_02x02_Counter_Clockwise
- added JP1: Jumper_2_Open, Connector_PinHeader_2.54mm:PinHeader_1x02_P2.54mm_Vertical, symbol Jumper:Jumper_2_Open
Connections:
- net Flash-MISO: now also J6.1 (Pin_1)
- net Flash-MOSI: now also J6.3 (Pin_3)
- net ICE_MISO: now also J6.4 (Pin_4)
- net ICE_MOSI: now also J6.2 (Pin_2)
- net ICE_SS_B: now also JP1.1 (A)
- net N25-CS: now also JP1.2 (B)
Changed lines of the file:
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@@
-    (stroke (width 0) (type default))
-  )
-  (wire (pts (xy 77.47 161.29) (xy 88.9 161.29))
     (stroke (width 0) (type default))
   )
@@
     (stroke (width 0) (type default))
   )
-  (wire (pts (xy 77.47 156.21) (xy 88.9 156.21))
-    (stroke (width 0) (type default))
-  )
   (wire (pts (xy 168.91 81.28) (xy 168.91 86.36))
     (stroke (width 0) (type default))
@@
     (stroke (width 0) (type default))
   )
-  (wire (pts (xy 57.15 158.75) (xy 67.31 158.75))
+  (wire (pts (xy 53.34 163.195) (xy 63.5 163.195))
     (stroke (width 0) (type default))
   )
@@
     (stroke (width 0) (type default))
   )
-  (wire (pts (xy 57.15 168.91) (xy 67.31 168.91))
+  (wire (pts (xy 53.34 165.735) (xy 63.5 165.735))
     (stroke (width 0) (type default))
   )
@@
     (stroke (width 0) (type default))
   )
+  (wire (pts (xy 140.335 116.84) (xy 144.78 116.84))
+    (stroke (width 0) (type default))
+  )
   (wire (pts (xy 73.66 71.12) (xy 83.82 71.12))
     (stroke (width 0) (type default))
@@
     (stroke (width 0) (type default))
   )
-  (wire (pts (xy 128.27 116.84) (xy 125.73 116.84))
+  (wire (pts (xy 125.73 116.84) (xy 130.175 116.84))
     (stroke (width 0) (type default))
   )
@@
     (stroke (width 0) (type default))
   )
-  (wire (pts (xy 77.47 171.45) (xy 88.9 171.45))
+  (wire (pts (xy 76.2 165.735) (xy 87.63 165.735))
     (stroke (width 0) (type default))
   )
@@
     (stroke (width 0) (type default))
   )
-  (wire (pts (xy 77.47 166.37) (xy 88.9 166.37))
+  (wire (pts (xy 76.2 163.195) (xy 87.63 163.195))
     (stroke (width 0) (type default))
   )
@@
   )
   (wire (pts (xy 68.58 63.5) (xy 73.66 63.5))
-    (stroke (width 0) (type default))
-  )
-  (wire (pts (xy 143.51 116.84) (xy 144.78 116.84))
     (stroke (width 0) (type default))
   )
@@
     (effects (font (size 1.27 1.27)) (justify left top))
   )
-  (label "ICE_MISO" (at 88.9 166.37 0) (fields_autoplaced)
+  (label "ICE_MISO" (at 87.63 163.195 0) (fields_autoplaced)
     (effects (font (size 1.27 1.27)) (justify left bottom))
   )
@@
     (effects (font (size 1.27 1.27)) (justify left bottom))
   )
-  (label "ICE_MOSI" (at 88.9 171.45 0) (fields_autoplaced)
-    (effects (font (size 1.27 1.27)) (justify left bottom))
-  )
-  (label "ICE_MISO" (at 88.9 161.29 0) (fields_autoplaced)
+  (label "ICE_MOSI" (at 53.34 165.735 0) (fields_autoplaced)
     (effects (font (size 1.27 1.27)) (justify left bottom))
   )
@@
   )
   (label "N25-HOLD" (at 176.53 114.3 0) (fields_autoplaced)
-    (effects (font (size 1.27 1.27)) (justify left bottom))
-  )
-  (label "ICE_MOSI" (at 88.9 156.21 0) (fields_autoplaced)
     (effects (font (size 1.27 1.27)) (justify left bottom))
   )
@@
     )
   )
-  (global_label "Flash-MOSI" (shape input) (at 57.15 158.75 180) (fields_autoplaced)
+  (global_label "Flash-MOSI" (shape input) (at 87.63 165.735 0) (fields_autoplaced)
+    (effects (font (size 1.27 1.27)) (justify left))
+    (property "Intersheetrefs" "${INTERSHEET_REFS}" (at 101.7843 165.735 0)
+      (effects (font (size 1.27 1.27)) (justify left) hide)
+    )
+  )
+  (global_label "Flash-MISO" (shape input) (at 53.34 163.195 180) (fields_autoplaced)
     (effects (font (size 1.27 1.27)) (justify right))
-    (property "Intersheetrefs" "${INTERSHEET_REFS}" (at 42.9957 158.75 0)
-      (effects (font (size 1.27 1.27)) (justify right) hide)
-    )
-  )
-  (global_label "Flash-MISO" (shape input) (at 57.15 168.91 180) (fields_autoplaced)
-    (effects (font (size 1.27 1.27)) (justify right))
-    (property "Intersheetrefs" "${INTERSHEET_REFS}" (at 42.9957 168.91 0)
+    (property "Intersheetrefs" "${INTERSHEET_REFS}" (at 39.1857 163.195 0)
       (effects (font (size 1.27 1.27)) (justify right) hide)
     )
@@
     )
   )
-  (symbol (lib_id "Switch:SW_DIP_x01") (at 135.89 116.84 0) (unit 1)
-    (in_bom yes) (on_board yes) (dnp no) (fields_autoplaced)
-    (property "Reference" "SW2" (at 135.89 111.2901 0)
-      (effects (font (size 1.27 1.27)))
-    )
-    (property "Value" "SW_DIP_x01" (at 135.89 113.2111 0)
-      (effects (font (size 1.27 1.27)))
-    )
-    (property "Footprint" "Button_Switch_SMD:SW_DIP_SPSTx01_Slide_9.78x4.72mm_W8.61mm_P2.54mm" (at 135.89 116.84 0)
-      (effects (font (size 1.27 1.27)) hide)
-    )
-    (property "Datasheet" "~" (at 135.89 116.84 0)
-      (effects (font (size 1.27 1.27)) hide)
-    )
-    (pin "1")
-    (pin "2")
-    (instances
-      (project "UFO-FPGA"
-        (path "/b3168f6a-c732-41d3-aeeb-d97dd2f1bb65/a9a0295d-b075-4952-a5ba-04debc5f691c"
-          (reference "SW2") (unit 1)
-        )
-        (path "/b3168f6a-c732-41d3-aeeb-d97dd2f1bb65/8a110dcf-7b5f-4510-96dd-3ef5ec8aca05"
-          (reference "SW4") (unit 1)
-        )
-      )
-    )
-  )
   (symbol (lib_id "Device:C") (at 130.81 53.34 0) (unit 1)
     (in_bom yes) (on_board yes) (dnp no) (fields_autoplaced)
@@
     )
   )
+  (symbol (lib_id "Connector_Generic:Conn_02x02_Counter_Clockwise") (at 68.58 163.195 0) (unit 1)
+    (in_bom yes) (on_board yes) (dnp no) (fields_autoplaced)
+    (property "Reference" "J6" (at 69.85 158.9151 0)
+      (effects (font (size 1.27 1.27)))
+    )
+    (property "Value" "Conn_02x02_Counter_Clockwise" (at 69.85 160.8361 0)
+      (effects (font (size 1.27 1.27)))
+    )
+    (property "Footprint" "Connector_PinHeader_2.54mm:PinHeader_2x02_P2.54mm_Vertical" (at 68.58 163.195 0)
+      (effects (font (size 1.27 1.27)) hide)
+    )
+    (property "Datasheet" "~" (at 68.58 163.195 0)
+      (effects (font (size 1.27 1.27)) hide)
+    )
+    (pin "1")
+    (pin "2")
+    (pin "3")
+    (pin "4")
+    (instances
+      (project "UFO-FPGA"
+        (path "/b3168f6a-c732-41d3-aeeb-d97dd2f1bb65/a9a0295d-b075-4952-a5ba-04debc5f691c"
+          (reference "J6") (unit 1)
+        )
+      )
+    )
+  )
   (symbol (lib_id "power:GND") (at 64.77 71.12 0) (unit 1)
     (in_bom yes) (on_board yes) (dnp no) (fields_autoplaced)
@@
         (path "/b3168f6a-c732-41d3-aeeb-d97dd2f1bb65/8a110dcf-7b5f-4510-96dd-3ef5ec8aca05"
           (reference "R40") (unit 1)
+        )
+      )
+    )
+  )
+  (symbol (lib_id "Jumper:Jumper_2_Open") (at 135.255 116.84 0) (unit 1)
+    (in_bom yes) (on_board yes) (dnp no) (fields_autoplaced)
+    (property "Reference" "JP1" (at 135.255 112.1791 0)
+      (effects (font (size 1.27 1.27)))
+    )
+    (property "Value" "Jumper_2_Open" (at 135.255 114.1001 0)
+      (effects (font (size 1.27 1.27)))
+    )
+    (property "Footprint" "Connector_PinHeader_2.54mm:PinHeader_1x02_P2.54mm_Vertical" (at 135.255 116.84 0)
+      (effects (font (size 1.27 1.27)) hide)
+    )
+    (property "Datasheet" "~" (at 135.255 116.84 0)
+      (effects (font (size 1.27 1.27)) hide)
+    )
+    (pin "1")
+    (pin "2")
+    (instances
+      (project "UFO-FPGA"
+        (path "/b3168f6a-c732-41d3-aeeb-d97dd2f1bb65/a9a0295d-b075-4952-a5ba-04debc5f691c"
+          (reference "JP1") (unit 1)
         )
       )
@@
         )
       )
-    )
-  )
-  (symbol (lib_id "Switch:SW_Push_DPDT") (at 72.39 163.83 0) (unit 1)
-    (in_bom yes) (on_board yes) (dnp no) (fields_autoplaced)
-    (property "Reference" "SW1" (at 72.39 152.8191 0)
-      (effects (font (size 1.27 1.27)))
-    )
-    (property "Value" "SW_Push_DPDT" (at 72.39 154.7401 0)
-      (effects (font (size 1.27 1.27)))
-    )
-    (property "Footprint" "Button_Switch_THT:SW_CuK_JS202011CQN_DPDT_Straight" (at 72.39 158.75 0)
-      (effects (font (size 1.27 1.27)) hide)
-    )
-    (property "Datasheet" "~" (at 72.39 158.75 0)
-      (effects (font (size 1.27 1.27)) hide)
-    )
-    (pin "1")
-    (pin "2")
-    (pin "3")
-    (pin "4")
-    (pin "5")
-    (pin "6")
-    (instances
-      (project "UFO-FPGA"
-        (path "/b3168f6a-c732-41d3-aeeb-d97dd2f1bb65/a9a0295d-b075-4952-a5ba-04debc5f691c"
-          (reference "SW1") (unit 1)
-        )
-        (path "/b3168f6a-c732-41d3-aeeb-d97dd2f1bb65/8a110dcf-7b5f-4510-96dd-3ef5ec8aca05"
-          (reference "SW3") (unit 1)
-        )
-      )

Commit message: pcb placement
Parts:
- removed TP1: TestPoint, TestPoint:TestPoint_Pad_1.5x1.5mm, symbol Connector:TestPoint
Changed lines of the file:
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@@
   (junction (at 63.5 77.47) (diameter 0) (color 0 0 0 0)
-  )
-  (junction (at 52.07 72.39) (diameter 0) (color 0 0 0 0)
   )
   (junction (at 83.82 71.12) (diameter 0) (color 0 0 0 0)
@@
     (stroke (width 0) (type default))
   )
-  (wire (pts (xy 52.07 72.39) (xy 52.07 77.47))
-    (stroke (width 0) (type default))
-  )
   (wire (pts (xy 115.57 107.95) (xy 147.32 107.95))
     (stroke (width 0) (type default))
@@
     (stroke (width 0) (type default))
   )
-  (wire (pts (xy 52.07 63.5) (xy 52.07 72.39))
+  (wire (pts (xy 52.07 63.5) (xy 52.07 77.47))
     (stroke (width 0) (type default))
   )
@@
         )
       )
-    )
-  )
-  (symbol (lib_id "Connector:TestPoint") (at 52.07 72.39 90) (mirror x) (unit 1)
-    (in_bom yes) (on_board yes) (dnp no)
-    (property "Reference" "TP1" (at 43.18 73.66 90)
-      (effects (font (size 1.27 1.27)))
-    )
-    (property "Value" "TestPoint" (at 43.18 71.12 90)
-      (effects (font (size 1.27 1.27)))
-    )
-    (property "Footprint" "TestPoint:TestPoint_Pad_1.5x1.5mm" (at 52.07 77.47 0)
-      (effects (font (size 1.27 1.27)) hide)
-    )
-    (property "Datasheet" "~" (at 52.07 77.47 0)
-      (effects (font (size 1.27 1.27)) hide)
-    )
-    (pin "1")
-    (instances
-      (project "UFO-FPGA"
-        (path "/b3168f6a-c732-41d3-aeeb-d97dd2f1bb65/6f7e0d88-d92b-4c4f-9dc8-64721cd46d41"
-          (reference "TP1") (unit 1)
-        )
-        (path "/b3168f6a-c732-41d3-aeeb-d97dd2f1bb65/a9a0295d-b075-4952-a5ba-04debc5f691c"
-          (reference "TP4") (unit 1)
-        )
-        (path "/b3168f6a-c732-41d3-aeeb-d97dd2f1bb65/8a110dcf-7b5f-4510-96dd-3ef5ec8aca05"
-          (reference "TP12") (unit 1)
-        )
-      )

Commit message: pcb
Connections:
- net ICE_MISO: now also J6.2 (Pin_2); no longer J6.4 (Pin_4)
- net ICE_MOSI: now also J6.4 (Pin_4); no longer J6.2 (Pin_2)
Changed lines of the file:
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@@
     (effects (font (size 1.27 1.27)) (justify left top))
   )
-  (label "ICE_MISO" (at 87.63 163.195 0) (fields_autoplaced)
+  (label "ICE_MISO" (at 53.34 165.735 0) (fields_autoplaced)
     (effects (font (size 1.27 1.27)) (justify left bottom))
   )
@@
     (effects (font (size 1.27 1.27)) (justify left bottom))
   )
-  (label "ICE_MOSI" (at 53.34 165.735 0) (fields_autoplaced)
+  (label "ICE_MOSI" (at 87.63 163.195 0) (fields_autoplaced)
     (effects (font (size 1.27 1.27)) (justify left bottom))
   )

Commit message: pcb 0603
Parts:
- C15, C16, C17, C20: footprint Capacitor_SMD:C_0805_2012Metric_Pad1.18x1.45mm_HandSolder -> Capacitor_SMD:C_0603_1608Metric_Pad1.08x0.95mm_HandSolder
Changed lines of the file:
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@@
       (effects (font (size 1.27 1.27)) (justify left))
     )
-    (property "Footprint" "Capacitor_SMD:C_0805_2012Metric_Pad1.18x1.45mm_HandSolder" (at 169.8752 81.28 0)
+    (property "Footprint" "Capacitor_SMD:C_0603_1608Metric_Pad1.08x0.95mm_HandSolder" (at 169.8752 81.28 0)
       (effects (font (size 1.27 1.27)) hide)
     )
@@
       (effects (font (size 1.27 1.27)) (justify left))
     )
-    (property "Footprint" "Capacitor_SMD:C_0805_2012Metric_Pad1.18x1.45mm_HandSolder" (at 84.7852 71.12 0)
+    (property "Footprint" "Capacitor_SMD:C_0603_1608Metric_Pad1.08x0.95mm_HandSolder" (at 84.7852 71.12 0)
       (effects (font (size 1.27 1.27)) hide)
     )
@@
       (effects (font (size 1.27 1.27)) (justify left))
     )
-    (property "Footprint" "Capacitor_SMD:C_0805_2012Metric_Pad1.18x1.45mm_HandSolder" (at 84.7852 81.28 0)
+    (property "Footprint" "Capacitor_SMD:C_0603_1608Metric_Pad1.08x0.95mm_HandSolder" (at 84.7852 81.28 0)
       (effects (font (size 1.27 1.27)) hide)
     )
@@
       (effects (font (size 1.27 1.27)) (justify left))
     )
-    (property "Footprint" "Capacitor_SMD:C_0805_2012Metric_Pad1.18x1.45mm_HandSolder" (at 131.7752 57.15 0)
-      (effects (font (size 1.27 1.27)) hide)
-    )
+    (property "Footprint" "Capacitor_SMD:C_0603_1608Metric_Pad1.08x0.95mm_HandSolder" (at 131.7752 57.15 0)
+      (effects (font (size 1.27 1.27)) hide)
+    )

Commit message: 0603
Parts:
- R21, R22, R23, R24: footprint Resistor_SMD:R_0805_2012Metric_Pad1.20x1.40mm_HandSolder -> Resistor_SMD:R_0603_1608Metric_Pad0.98x0.95mm_HandSolder
Changed lines of the file:
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@@
       (effects (font (size 1.27 1.27)) (justify left))
     )
-    (property "Footprint" "Resistor_SMD:R_0805_2012Metric_Pad1.20x1.40mm_HandSolder" (at 211.582 60.96 90)
+    (property "Footprint" "Resistor_SMD:R_0603_1608Metric_Pad0.98x0.95mm_HandSolder" (at 211.582 60.96 90)
       (effects (font (size 1.27 1.27)) hide)
     )
@@
       (effects (font (size 1.27 1.27)) (justify left))
     )
-    (property "Footprint" "Resistor_SMD:R_0805_2012Metric_Pad1.20x1.40mm_HandSolder" (at 219.202 60.96 90)
+    (property "Footprint" "Resistor_SMD:R_0603_1608Metric_Pad0.98x0.95mm_HandSolder" (at 219.202 60.96 90)
       (effects (font (size 1.27 1.27)) hide)
     )
@@
       (effects (font (size 1.27 1.27)) (justify left))
     )
-    (property "Footprint" "Resistor_SMD:R_0805_2012Metric_Pad1.20x1.40mm_HandSolder" (at 203.962 60.96 90)
+    (property "Footprint" "Resistor_SMD:R_0603_1608Metric_Pad0.98x0.95mm_HandSolder" (at 203.962 60.96 90)
       (effects (font (size 1.27 1.27)) hide)
     )
@@
       (effects (font (size 1.27 1.27)) (justify left))
     )
-    (property "Footprint" "Resistor_SMD:R_0805_2012Metric_Pad1.20x1.40mm_HandSolder" (at 145.542 53.34 90)
-      (effects (font (size 1.27 1.27)) hide)
-    )
+    (property "Footprint" "Resistor_SMD:R_0603_1608Metric_Pad0.98x0.95mm_HandSolder" (at 145.542 53.34 90)
+      (effects (font (size 1.27 1.27)) hide)
+    )

Commit message: pcb
added John zendong
Parts:
- removed U1: ICE40HX8K-BG121, Package_BGA:BGA-121_9.0x9.0mm_Layout11x11_P0.8mm_Ball0.4mm_Pad0.35mm_NSMD, symbol FPGA_Lattice:ICE40HX8K-BG121
- added U4: ICE40HX4K-TQ144, Package_QFP:TQFP-144_20x20mm_P0.5mm, symbol FPGA_Lattice:ICE40HX4K-TQ144
- J6: footprint Connector_PinHeader_2.54mm:PinHeader_2x02_P2.54mm_Vertical -> Connector_PinHeader_1.27mm:PinHeader_2x02_P1.27mm_Vertical
- JP1: footprint Connector_PinHeader_2.54mm:PinHeader_1x02_P2.54mm_Vertical -> Connector_PinHeader_1.27mm:PinHeader_1x02_P1.27mm_Vertical
Connections:
- net +1V2: now also U4.111 (VCC), U4.27 (VCC), U4.40 (VCC), U4.92 (VCC)
- net +2V5: now also U4.108 (VPP_2V5)
- net +3V3: now also U4.72 (VCC_SPI)
- net GND: now also U4.103 (GND), U4.127 (GNDPLL1), U4.13 (GND), U4.132 (GND), U4.14 (GND), U4.140 (GND), U4.5 (GND), U4.53 (GNDPLL0), U4.59 (GND), U4.69 (GND), U4.86 (GND)
- net ICE_MISO: now also U4.67 (IOB_105_SDO)
- net ICE_MOSI: now also U4.68 (IOB_106_SDI)
- net ICE_SCK: now also U4.70 (IOB_107_SCK)
- net ICE_SS_B: now also U4.71 (IOB_108_SS)
- net VCCPLL0: now also U4.54 (VCCPLL0)
- net VCCPLL1: now also U4.126 (VCCPLL1)
- new net ICE_CDONE: U4.65 (CDONE)
- new net ICE_CREST: U4.66 (~{CRESET})
Other:
- moved on the sheet: C17, C18, C19, C20, R25, R26, TP1
