File: UFO-FPGA/BANK4.kicad_sch (KiCad schematic)
At the start: 19 parts, among them J6 Conn_02x02_Counter_Clockwise, U4 ICE40HX4K-TQ144, U9 N25Q032A13ESC40F

Commit message: pcb
Parts:
- U9: footprint Package_SO:SOP-8_3.9x4.9mm_P1.27mm -> Package_SO:SSOP-8_5.25x5.24mm_P1.27mm
Changed lines of the file:
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@@
       (effects (font (size 1.27 1.27)) (justify left))
     )
-    (property "Footprint" "Package_SO:SOP-8_3.9x4.9mm_P1.27mm" (at 146.05 121.285 0)
+    (property "Footprint" "Package_SO:SSOP-8_5.25x5.24mm_P1.27mm" (at 146.05 121.285 0)
       (effects (font (size 1.27 1.27)) hide)
     )

Commit message: pcb
Parts:
- C15, C17, C20: footprint Capacitor_SMD:C_0603_1608Metric_Pad1.08x0.95mm_HandSolder -> Capacitor_SMD:C_0805_2012Metric_Pad1.18x1.45mm_HandSolder
- TP1: footprint TestPoint:TestPoint_Pad_1.5x1.5mm -> TestPoint:TestPoint_Pad_1.0x1.0mm
Changed lines of the file:
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@@
       (effects (font (size 1.27 1.27)) (justify left))
     )
-    (property "Footprint" "Capacitor_SMD:C_0603_1608Metric_Pad1.08x0.95mm_HandSolder" (at 169.8752 81.28 0)
+    (property "Footprint" "Capacitor_SMD:C_0805_2012Metric_Pad1.18x1.45mm_HandSolder" (at 169.8752 81.28 0)
       (effects (font (size 1.27 1.27)) hide)
     )
@@
       (effects (font (size 1.27 1.27)) (justify left))
     )
-    (property "Footprint" "Capacitor_SMD:C_0603_1608Metric_Pad1.08x0.95mm_HandSolder" (at 82.2452 82.55 0)
+    (property "Footprint" "Capacitor_SMD:C_0805_2012Metric_Pad1.18x1.45mm_HandSolder" (at 82.2452 82.55 0)
       (effects (font (size 1.27 1.27)) hide)
     )
@@
       (effects (font (size 1.27 1.27)) (justify left))
     )
-    (property "Footprint" "Capacitor_SMD:C_0603_1608Metric_Pad1.08x0.95mm_HandSolder" (at 82.2452 69.85 0)
+    (property "Footprint" "Capacitor_SMD:C_0805_2012Metric_Pad1.18x1.45mm_HandSolder" (at 82.2452 69.85 0)
       (effects (font (size 1.27 1.27)) hide)
     )
@@
       (effects (font (size 1.27 1.27)) (justify left))
     )
-    (property "Footprint" "TestPoint:TestPoint_Pad_1.5x1.5mm" (at 60.96 74.93 0)
+    (property "Footprint" "TestPoint:TestPoint_Pad_1.0x1.0mm" (at 60.96 74.93 0)
       (effects (font (size 1.27 1.27)) hide)
     )
@@
       (effects (font (size 1.27 1.27)) (justify right))
     )
-    (property "Footprint" "TestPoint:TestPoint_Pad_1.5x1.5mm" (at 55.88 66.04 0)
-      (effects (font (size 1.27 1.27)) hide)
-    )
+    (property "Footprint" "TestPoint:TestPoint_Pad_1.0x1.0mm" (at 55.88 66.04 0)
+      (effects (font (size 1.27 1.27)) hide)
+    )

Commit message: pcb
added monkey
Changed lines of the file:
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@@
     (company "Universal-Field-Objects")
   )
+  (junction (at 125.73 116.84) (diameter 0) (color 0 0 0 0)
+  )
   (junction (at 130.81 40.64) (diameter 0) (color 0 0 0 0)
   )
@@
   )
   (junction (at 81.28 69.85) (diameter 0) (color 0 0 0 0)
-  )
-  (junction (at 126.238 116.84) (diameter 0) (color 0 0 0 0)
   )
   (junction (at 220.98 40.64) (diameter 0) (color 0 0 0 0)
@@
     (stroke (width 0) (type default))
   )
-  (wire (pts (xy 115.57 116.84) (xy 126.238 116.84))
-    (stroke (width 0) (type default))
-  )
-  (wire (pts (xy 126.238 100.33) (xy 126.238 116.84))
-    (stroke (width 0) (type default))
-  )
   (wire (pts (xy 213.36 40.64) (xy 213.36 57.15))
     (stroke (width 0) (type default))
@@
     (stroke (width 0) (type default))
   )
-  (wire (pts (xy 143.002 76.2) (xy 143.002 100.33))
-    (stroke (width 0) (type default))
-  )
   (wire (pts (xy 205.74 40.64) (xy 205.74 57.15))
     (stroke (width 0) (type default))
@@
     (stroke (width 0) (type default))
   )
-  (wire (pts (xy 124.46 76.2) (xy 143.002 76.2))
+  (wire (pts (xy 124.46 76.2) (xy 144.78 76.2))
     (stroke (width 0) (type default))
   )
@@
     (stroke (width 0) (type default))
   )
+  (wire (pts (xy 125.73 116.84) (xy 130.175 116.84))
+    (stroke (width 0) (type default))
+  )
   (wire (pts (xy 144.78 116.84) (xy 152.4 116.84))
     (stroke (width 0) (type default))
@@
     (stroke (width 0) (type default))
   )
-  (wire (pts (xy 126.238 116.84) (xy 130.175 116.84))
+  (wire (pts (xy 115.57 116.84) (xy 125.73 116.84))
     (stroke (width 0) (type default))
   )
@@
     (stroke (width 0) (type default))
   )
-  (wire (pts (xy 143.002 100.33) (xy 126.238 100.33))
+  (wire (pts (xy 125.73 100.33) (xy 144.78 100.33))
     (stroke (width 0) (type default))
   )
@@
     (stroke (width 0) (type default))
   )
+  (wire (pts (xy 144.78 76.2) (xy 144.78 100.33))
+    (stroke (width 0) (type default))
+  )
   (wire (pts (xy 71.12 69.85) (xy 77.47 69.85))
     (stroke (width 0) (type default))
@@
     (stroke (width 0) (type default))
   )
+  (wire (pts (xy 125.73 116.84) (xy 125.73 100.33))
+    (stroke (width 0) (type default))
+  )

Commit message: pcb silkscreen
Parts:
- J6: footprint Connector_PinHeader_1.27mm:PinHeader_2x02_P1.27mm_Vertical -> Connector_PinHeader_2.00mm:PinHeader_2x02_P2.00mm_Vertical
- JP1: footprint Connector_PinHeader_1.27mm:PinHeader_1x02_P1.27mm_Vertical -> Connector_PinHeader_2.00mm:PinHeader_1x02_P2.00mm_Vertical
Connections:
- net Flash-MOSI: now also J6.4 (Pin_4); no longer J6.3 (Pin_3)
- net ICE_MOSI: now also J6.3 (Pin_3); no longer J6.4 (Pin_4)
Changed lines of the file:
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@@
+    (stroke (width 0) (type default))
+  )
+  (wire (pts (xy 76.2 165.735) (xy 87.63 165.735))
     (stroke (width 0) (type default))
   )
@@
     (stroke (width 0) (type default))
   )
+  (wire (pts (xy 168.91 73.66) (xy 168.91 69.85))
+    (stroke (width 0) (type default))
+  )
+  (wire (pts (xy 205.74 64.77) (xy 205.74 114.3))
+    (stroke (width 0) (type default))
+  )
+  (wire (pts (xy 115.57 107.95) (xy 147.32 107.95))
+    (stroke (width 0) (type default))
+  )
+  (wire (pts (xy 162.56 69.85) (xy 162.56 100.33))
+    (stroke (width 0) (type default))
+  )
+  (wire (pts (xy 77.47 69.85) (xy 81.28 69.85))
+    (stroke (width 0) (type default))
+  )
+  (wire (pts (xy 144.78 133.35) (xy 220.98 133.35))
+    (stroke (width 0) (type default))
+  )
+  (wire (pts (xy 115.57 116.84) (xy 125.73 116.84))
+    (stroke (width 0) (type default))
+  )
+  (wire (pts (xy 147.32 128.27) (xy 147.32 114.3))
+    (stroke (width 0) (type default))
+  )
+  (wire (pts (xy 71.12 82.55) (xy 62.23 82.55))
+    (stroke (width 0) (type default))
+  )
+  (wire (pts (xy 81.28 82.55) (xy 91.44 82.55))
+    (stroke (width 0) (type default))
+  )
+  (wire (pts (xy 130.81 40.64) (xy 147.32 40.64))
+    (stroke (width 0) (type default))
+  )
+  (wire (pts (xy 147.32 107.95) (xy 152.4 107.95))
+    (stroke (width 0) (type default))
+  )
+  (wire (pts (xy 49.53 66.04) (xy 49.53 74.93))
+    (stroke (width 0) (type default))
+  )
+  (wire (pts (xy 168.91 69.85) (xy 162.56 69.85))
+    (stroke (width 0) (type default))
+  )
+  (wire (pts (xy 109.22 48.895) (xy 109.22 50.8))
+    (stroke (width 0) (type default))
+  )
+  (wire (pts (xy 140.335 116.84) (xy 144.78 116.84))
+    (stroke (width 0) (type default))
+  )
+  (wire (pts (xy 71.12 82.55) (xy 81.28 82.55))
+    (stroke (width 0) (type default))
+  )
+  (wire (pts (xy 147.32 114.3) (xy 152.4 114.3))
+    (stroke (width 0) (type default))
+  )
+  (wire (pts (xy 125.73 100.33) (xy 144.78 100.33))
+    (stroke (width 0) (type default))
+  )
+  (wire (pts (xy 162.56 123.19) (xy 162.56 124.46))
+    (stroke (width 0) (type default))
+  )
+  (wire (pts (xy 109.22 48.26) (xy 109.22 48.895))
+    (stroke (width 0) (type default))
+  )
+  (wire (pts (xy 71.12 74.93) (xy 81.28 74.93))
+    (stroke (width 0) (type default))
+  )
+  (wire (pts (xy 162.56 40.64) (xy 162.56 69.85))
+    (stroke (width 0) (type default))
+  )
+  (wire (pts (xy 60.96 66.04) (xy 66.04 66.04))
+    (stroke (width 0) (type default))
+  )
+  (wire (pts (xy 124.46 71.12) (xy 135.89 71.12))
+    (stroke (width 0) (type default))
+  )
+  (wire (pts (xy 124.46 68.58) (xy 135.89 68.58))
+    (stroke (width 0) (type default))
+  )
+  (wire (pts (xy 116.84 40.64) (xy 116.84 53.34))
+    (stroke (width 0) (type default))
+  )
+  (wire (pts (xy 144.78 76.2) (xy 144.78 100.33))
+    (stroke (width 0) (type default))
+  )
+  (wire (pts (xy 71.12 69.85) (xy 77.47 69.85))
+    (stroke (width 0) (type default))
+  )
+  (wire (pts (xy 109.22 40.64) (xy 116.84 40.64))
+    (stroke (width 0) (type default))
+  )
+  (wire (pts (xy 76.2 163.195) (xy 87.63 163.195))
+    (stroke (width 0) (type default))
+  )
+  (wire (pts (xy 172.72 105.41) (xy 180.34 105.41))
+    (stroke (width 0) (type default))
+  )
   (wire (pts (xy 53.34 165.735) (xy 63.5 165.735))
-    (stroke (width 0) (type default))
-  )
-  (wire (pts (xy 168.91 73.66) (xy 168.91 69.85))
-    (stroke (width 0) (type default))
-  )
-  (wire (pts (xy 205.74 64.77) (xy 205.74 114.3))
-    (stroke (width 0) (type default))
-  )
-  (wire (pts (xy 115.57 107.95) (xy 147.32 107.95))
-    (stroke (width 0) (type default))
-  )
-  (wire (pts (xy 162.56 69.85) (xy 162.56 100.33))
-    (stroke (width 0) (type default))
-  )
-  (wire (pts (xy 77.47 69.85) (xy 81.28 69.85))
-    (stroke (width 0) (type default))
-  )
-  (wire (pts (xy 144.78 133.35) (xy 220.98 133.35))
-    (stroke (width 0) (type default))
-  )
-  (wire (pts (xy 115.57 116.84) (xy 125.73 116.84))
-    (stroke (width 0) (type default))
-  )
-  (wire (pts (xy 147.32 128.27) (xy 147.32 114.3))
-    (stroke (width 0) (type default))
-  )
-  (wire (pts (xy 71.12 82.55) (xy 62.23 82.55))
-    (stroke (width 0) (type default))
-  )
-  (wire (pts (xy 81.28 82.55) (xy 91.44 82.55))
-    (stroke (width 0) (type default))
-  )
-  (wire (pts (xy 130.81 40.64) (xy 147.32 40.64))
-    (stroke (width 0) (type default))
-  )
-  (wire (pts (xy 147.32 107.95) (xy 152.4 107.95))
-    (stroke (width 0) (type default))
-  )
-  (wire (pts (xy 49.53 66.04) (xy 49.53 74.93))
-    (stroke (width 0) (type default))
-  )
-  (wire (pts (xy 168.91 69.85) (xy 162.56 69.85))
-    (stroke (width 0) (type default))
-  )
-  (wire (pts (xy 109.22 48.895) (xy 109.22 50.8))
-    (stroke (width 0) (type default))
-  )
-  (wire (pts (xy 140.335 116.84) (xy 144.78 116.84))
-    (stroke (width 0) (type default))
-  )
-  (wire (pts (xy 71.12 82.55) (xy 81.28 82.55))
-    (stroke (width 0) (type default))
-  )
-  (wire (pts (xy 147.32 114.3) (xy 152.4 114.3))
-    (stroke (width 0) (type default))
-  )
-  (wire (pts (xy 125.73 100.33) (xy 144.78 100.33))
-    (stroke (width 0) (type default))
-  )
-  (wire (pts (xy 162.56 123.19) (xy 162.56 124.46))
-    (stroke (width 0) (type default))
-  )
-  (wire (pts (xy 109.22 48.26) (xy 109.22 48.895))
-    (stroke (width 0) (type default))
-  )
-  (wire (pts (xy 71.12 74.93) (xy 81.28 74.93))
-    (stroke (width 0) (type default))
-  )
-  (wire (pts (xy 162.56 40.64) (xy 162.56 69.85))
-    (stroke (width 0) (type default))
-  )
-  (wire (pts (xy 60.96 66.04) (xy 66.04 66.04))
-    (stroke (width 0) (type default))
-  )
-  (wire (pts (xy 124.46 71.12) (xy 135.89 71.12))
-    (stroke (width 0) (type default))
-  )
-  (wire (pts (xy 124.46 68.58) (xy 135.89 68.58))
-    (stroke (width 0) (type default))
-  )
-  (wire (pts (xy 116.84 40.64) (xy 116.84 53.34))
-    (stroke (width 0) (type default))
-  )
-  (wire (pts (xy 144.78 76.2) (xy 144.78 100.33))
-    (stroke (width 0) (type default))
-  )
-  (wire (pts (xy 71.12 69.85) (xy 77.47 69.85))
-    (stroke (width 0) (type default))
-  )
-  (wire (pts (xy 76.2 165.735) (xy 87.63 165.735))
-    (stroke (width 0) (type default))
-  )
-  (wire (pts (xy 109.22 40.64) (xy 116.84 40.64))
-    (stroke (width 0) (type default))
-  )
-  (wire (pts (xy 76.2 163.195) (xy 87.63 163.195))
-    (stroke (width 0) (type default))
-  )
-  (wire (pts (xy 172.72 105.41) (xy 180.34 105.41))
     (stroke (width 0) (type default))
   )
@@
     (effects (font (size 1.27 1.27)) (justify left bottom))
   )
-  (label "ICE_MOSI" (at 87.63 163.195 0) (fields_autoplaced)
-    (effects (font (size 1.27 1.27)) (justify left bottom))
+  (label "ICE_MOSI" (at 87.63 165.735 180) (fields_autoplaced)
+    (effects (font (size 1.27 1.27)) (justify right bottom))
   )
   (label "N25-CS" (at 149.225 133.35 0) (fields_autoplaced)
@@
     )
   )
-  (global_label "Flash-MOSI" (shape input) (at 87.63 165.735 0) (fields_autoplaced)
+  (global_label "Flash-MOSI" (shape input) (at 87.63 163.195 0) (fields_autoplaced)
     (effects (font (size 1.27 1.27)) (justify left))
-    (property "Intersheetrefs" "${INTERSHEET_REFS}" (at 101.7843 165.735 0)
+    (property "Intersheetrefs" "${INTERSHEET_REFS}" (at 101.7843 163.195 0)
       (effects (font (size 1.27 1.27)) (justify left) hide)
     )
@@
       (effects (font (size 1.27 1.27)))
     )
-    (property "Footprint" "Connector_PinHeader_1.27mm:PinHeader_2x02_P1.27mm_Vertical" (at 68.58 163.195 0)
+    (property "Footprint" "Connector_PinHeader_2.00mm:PinHeader_2x02_P2.00mm_Vertical" (at 68.58 163.195 0)
       (effects (font (size 1.27 1.27)) hide)
     )
@@
       (effects (font (size 1.27 1.27)))
     )
-    (property "Footprint" "Connector_PinHeader_1.27mm:PinHeader_1x02_P1.27mm_Vertical" (at 135.255 116.84 0)
-      (effects (font (size 1.27 1.27)) hide)
-    )
+    (property "Footprint" "Connector_PinHeader_2.00mm:PinHeader_1x02_P2.00mm_Vertical" (at 135.255 116.84 0)
+      (effects (font (size 1.27 1.27)) hide)
+    )
