File: UFO-FPGA/Programmer.kicad_sch (KiCad schematic)
At the start: 41 parts, among them U2 FT2232HL, U3 ASDMB-12MHz, U5 93LC56CT-I/MS

Commit message: Vregout
Connections:
- net +1V8: now also U2.49 (VREGOUT)
Changed lines of the file:
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@@
   (junction (at 184.785 26.035) (diameter 0) (color 0 0 0 0)
   )
+  (junction (at 183.515 86.36) (diameter 0) (color 0 0 0 0)
+  )
   (junction (at 166.37 26.035) (diameter 0) (color 0 0 0 0)
   )
@@
   (junction (at 323.85 154.94) (diameter 0) (color 0 0 0 0)
   )
-  (junction (at 183.515 86.36) (diameter 0) (color 0 0 0 0)
-  )
   (junction (at 220.345 193.04) (diameter 0) (color 0 0 0 0)
   )
@@
   )
   (junction (at 127 129.54) (diameter 0) (color 0 0 0 0)
+  )
+  (junction (at 183.515 90.805) (diameter 0) (color 0 0 0 0)
   )
   (junction (at 246.38 193.04) (diameter 0) (color 0 0 0 0)
@@
     (stroke (width 0) (type default))
   )
+  (wire (pts (xy 183.515 86.36) (xy 223.52 86.36))
+    (stroke (width 0) (type default))
+  )
   (wire (pts (xy 243.84 193.04) (xy 246.38 193.04))
     (stroke (width 0) (type default))
@@
     (stroke (width 0) (type default))
   )
-  (wire (pts (xy 183.515 86.36) (xy 183.515 99.06))
+  (wire (pts (xy 183.515 78.74) (xy 183.515 86.36))
     (stroke (width 0) (type default))
   )
@@
     (stroke (width 0) (type default))
   )
-  (wire (pts (xy 185.674 86.36) (xy 183.515 86.36))
-    (stroke (width 0) (type default))
-  )
   (wire (pts (xy 295.91 162.56) (xy 302.26 162.56))
     (stroke (width 0) (type default))
@@
     (stroke (width 0) (type default))
   )
-  (wire (pts (xy 183.515 78.74) (xy 183.515 86.36))
-    (stroke (width 0) (type default))
-  )
   (wire (pts (xy 140.335 152.4) (xy 223.52 152.4))
     (stroke (width 0) (type default))
@@
     (stroke (width 0) (type default))
   )
+  (wire (pts (xy 183.515 86.36) (xy 183.515 90.805))
+    (stroke (width 0) (type default))
+  )
   (wire (pts (xy 256.54 193.04) (xy 259.08 193.04))
     (stroke (width 0) (type default))
@@
     (stroke (width 0) (type default))
   )
+  (wire (pts (xy 183.515 90.805) (xy 185.42 90.805))
+    (stroke (width 0) (type default))
+  )
   (wire (pts (xy 246.38 193.04) (xy 248.92 193.04))
     (stroke (width 0) (type default))
@@
   )
   (wire (pts (xy 309.88 154.94) (xy 312.42 154.94))
+    (stroke (width 0) (type default))
+  )
+  (wire (pts (xy 183.515 90.805) (xy 183.515 99.06))
     (stroke (width 0) (type default))
   )
@@
     )
   )
-  (symbol (lib_id "power:PWR_FLAG") (at 185.674 86.36 270) (mirror x) (unit 1)
+  (symbol (lib_id "power:PWR_FLAG") (at 185.42 90.805 270) (mirror x) (unit 1)
     (in_bom yes) (on_board yes) (dnp no) (fields_autoplaced)
-    (property "Reference" "#FLG01" (at 187.579 86.36 0)
+    (property "Reference" "#FLG01" (at 187.325 90.805 0)
       (effects (font (size 1.27 1.27)) hide)
     )
-    (property "Value" "PWR_FLAG" (at 188.8489 86.6768 90)
+    (property "Value" "PWR_FLAG" (at 188.5949 91.1218 90)
       (effects (font (size 1.27 1.27)) (justify left))
     )
-    (property "Footprint" "" (at 185.674 86.36 0)
+    (property "Footprint" "" (at 185.42 90.805 0)
       (effects (font (size 1.27 1.27)) hide)
     )
-    (property "Datasheet" "~" (at 185.674 86.36 0)
+    (property "Datasheet" "~" (at 185.42 90.805 0)
       (effects (font (size 1.27 1.27)) hide)
     )

Commit message: PCB
Connections:
- net FLASH-MISO renamed FLASH_MISO
- net FLASH-MOSI renamed FLASH_MOSI
Other:
- moved on the sheet: R7
Changed lines of the file:
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@@
   (junction (at 127 129.54) (diameter 0) (color 0 0 0 0)
-  )
-  (junction (at 183.515 90.805) (diameter 0) (color 0 0 0 0)
   )
   (junction (at 246.38 193.04) (diameter 0) (color 0 0 0 0)
@@
     (stroke (width 0) (type default))
   )
-  (wire (pts (xy 177.8 185.42) (xy 177.8 191.262))
-    (stroke (width 0) (type default))
-  )
   (wire (pts (xy 259.08 64.135) (xy 259.08 73.66))
     (stroke (width 0) (type default))
@@
     (stroke (width 0) (type default))
   )
+  (wire (pts (xy 177.8 185.42) (xy 177.8 191.77))
+    (stroke (width 0) (type default))
+  )
   (wire (pts (xy 184.785 26.035) (xy 184.785 29.21))
     (stroke (width 0) (type default))
@@
     (stroke (width 0) (type default))
   )
+  (wire (pts (xy 177.8 191.77) (xy 180.975 191.77))
+    (stroke (width 0) (type default))
+  )
   (wire (pts (xy 212.09 119.38) (xy 223.52 119.38))
     (stroke (width 0) (type default))
@@
     (stroke (width 0) (type default))
   )
+  (wire (pts (xy 188.595 191.77) (xy 191.77 191.77))
+    (stroke (width 0) (type default))
+  )
   (wire (pts (xy 166.37 26.035) (xy 175.26 26.035))
     (stroke (width 0) (type default))
@@
     (stroke (width 0) (type default))
   )
-  (wire (pts (xy 190.5 191.262) (xy 192.024 191.262))
-    (stroke (width 0) (type default))
-  )
   (wire (pts (xy 203.2 40.005) (xy 203.2 36.83))
     (stroke (width 0) (type default))
@@
     (stroke (width 0) (type default))
   )
-  (wire (pts (xy 183.515 86.36) (xy 183.515 90.805))
+  (wire (pts (xy 183.515 86.36) (xy 183.515 99.06))
     (stroke (width 0) (type default))
   )
@@
     (stroke (width 0) (type default))
   )
-  (wire (pts (xy 177.8 191.262) (xy 182.88 191.262))
-    (stroke (width 0) (type default))
-  )
   (wire (pts (xy 254 58.42) (xy 254 64.135))
     (stroke (width 0) (type default))
@@
     (stroke (width 0) (type default))
   )
-  (wire (pts (xy 183.515 90.805) (xy 185.42 90.805))
-    (stroke (width 0) (type default))
-  )
   (wire (pts (xy 246.38 193.04) (xy 248.92 193.04))
     (stroke (width 0) (type default))
@@
   )
   (wire (pts (xy 309.88 154.94) (xy 312.42 154.94))
-    (stroke (width 0) (type default))
-  )
-  (wire (pts (xy 183.515 90.805) (xy 183.515 99.06))
     (stroke (width 0) (type default))
   )
@@
     (effects (font (size 1.27 1.27)) (justify right bottom))
   )
-  (label "FLASH-MISO" (at 287.655 86.36 0) (fields_autoplaced)
-    (effects (font (size 1.27 1.27)) (justify left bottom))
-  )
-  (label "FLASH-MOSI" (at 287.655 83.82 0) (fields_autoplaced)
+  (label "FLASH_MISO" (at 287.655 86.36 0) (fields_autoplaced)
+    (effects (font (size 1.27 1.27)) (justify left bottom))
+  )
+  (label "FLASH_MOSI" (at 287.655 83.82 0) (fields_autoplaced)
     (effects (font (size 1.27 1.27)) (justify left bottom))
   )
@@
     )
   )
-  (global_label "ICE_CLK" (shape input) (at 192.024 191.262 0) (fields_autoplaced)
+  (global_label "ICE_CLK" (shape input) (at 191.77 191.77 0) (fields_autoplaced)
     (effects (font (size 1.27 1.27)) (justify left))
-    (property "Intersheetrefs" "${INTERSHEET_REFS}" (at 202.4893 191.262 0)
+    (property "Intersheetrefs" "${INTERSHEET_REFS}" (at 202.2353 191.77 0)
       (effects (font (size 1.27 1.27)) (justify left) hide)
     )
@@
     )
   )
-  (symbol (lib_id "power:PWR_FLAG") (at 185.42 90.805 270) (mirror x) (unit 1)
-    (in_bom yes) (on_board yes) (dnp no) (fields_autoplaced)
-    (property "Reference" "#FLG01" (at 187.325 90.805 0)
-      (effects (font (size 1.27 1.27)) hide)
-    )
-    (property "Value" "PWR_FLAG" (at 188.5949 91.1218 90)
-      (effects (font (size 1.27 1.27)) (justify left))
-    )
-    (property "Footprint" "" (at 185.42 90.805 0)
-      (effects (font (size 1.27 1.27)) hide)
-    )
-    (property "Datasheet" "~" (at 185.42 90.805 0)
-      (effects (font (size 1.27 1.27)) hide)
-    )
-    (pin "1")
-    (instances
-      (project "UFO-FPGA"
-        (path "/b3168f6a-c732-41d3-aeeb-d97dd2f1bb65/eec89a79-dace-443c-aa86-713b48a49f95"
-          (reference "#FLG01") (unit 1)
-        )
-      )
-    )
-  )
   (symbol (lib_id "Device:R") (at 307.34 142.24 270) (mirror x) (unit 1)
     (in_bom yes) (on_board yes) (dnp no)
@@
     )
   )
-  (symbol (lib_id "Device:R") (at 186.69 191.262 90) (unit 1)
-    (in_bom yes) (on_board yes) (dnp no)
-    (property "Reference" "R7" (at 186.69 195.2879 90)
-      (effects (font (size 1.27 1.27)))
-    )
-    (property "Value" "0" (at 186.69 193.3669 90)
-      (effects (font (size 1.27 1.27)))
-    )
-    (property "Footprint" "Resistor_SMD:R_0805_2012Metric_Pad1.20x1.40mm_HandSolder" (at 186.69 193.04 90)
-      (effects (font (size 1.27 1.27)) hide)
-    )
-    (property "Datasheet" "~" (at 186.69 191.262 0)
-      (effects (font (size 1.27 1.27)) hide)
-    )
+  (symbol (lib_id "Device:R") (at 184.785 191.77 90) (unit 1)
+    (in_bom yes) (on_board yes) (dnp no)
+    (property "Reference" "R7" (at 184.785 195.7959 90)
+      (effects (font (size 1.27 1.27)))
+    )
+    (property "Value" "0" (at 184.785 193.8749 90)
+      (effects (font (size 1.27 1.27)))
+    )
+    (property "Footprint" "Resistor_SMD:R_0805_2012Metric_Pad1.20x1.40mm_HandSolder" (at 184.785 193.548 90)
+      (effects (font (size 1.27 1.27)) hide)
+    )
+    (property "Datasheet" "~" (at 184.785 191.77 0)
+      (effects (font (size 1.27 1.27)) hide)
+    )

Commit message: PCB
many pcb changes
-started routing
-added vias
-power planes
-ground planes
Parts:
- removed C14, C5, C6: 100nF, Capacitor_SMD:C_0805_2012Metric_Pad1.18x1.45mm_HandSolder, symbol Device:C
- C2, C3, C4: value 100nF -> 200nF
Connections:
- net rxled-mid: now reaches R33.1, RXLED1.2 (A)
- net ftd-ref: now reaches R6.1, U2.6 (REF)
- net txled out: now reaches TXLED1.1 (K), U2.55 (BCBUS4)
- net txled-mid: now reaches R34.1, TXLED1.2 (A)
- net ftd-reset: now reaches R5.1, U2.14 (~{RESET})
- net rxled out: now reaches RXLED1.1 (K), U2.54 (BCBUS3)
Other:
- moved on the sheet: C2, C3, C4, R33, R34

Commit message: pcb prog redesign
Connections:
- net DM renamed D-
- net DP renamed D+
Changed lines of the file:
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@@
     )
   )
-  (global_label "DP" (shape input) (at 215.265 109.22 180) (fields_autoplaced)
+  (global_label "D+" (shape input) (at 215.265 109.22 180) (fields_autoplaced)
     (effects (font (size 1.27 1.27)) (justify right))
-    (property "Intersheetrefs" "${INTERSHEET_REFS}" (at 209.8192 109.22 0)
+    (property "Intersheetrefs" "${INTERSHEET_REFS}" (at 209.5168 109.22 0)
       (effects (font (size 1.27 1.27)) (justify right) hide)
     )
@@
     )
   )
-  (global_label "DM" (shape input) (at 215.265 106.68 180) (fields_autoplaced)
+  (global_label "D-" (shape input) (at 215.265 106.68 180) (fields_autoplaced)
     (effects (font (size 1.27 1.27)) (justify right))
-    (property "Intersheetrefs" "${INTERSHEET_REFS}" (at 209.6378 106.68 0)
+    (property "Intersheetrefs" "${INTERSHEET_REFS}" (at 209.5168 106.68 0)
       (effects (font (size 1.27 1.27)) (justify right) hide)
     )

Commit message: pcb 0603
Parts:
- C1, C12, C13, C2, C3, C4, C7, C8: footprint Capacitor_SMD:C_0805_2012Metric_Pad1.18x1.45mm_HandSolder -> Capacitor_SMD:C_0603_1608Metric_Pad1.08x0.95mm_HandSolder
Changed lines of the file:
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@@
       (effects (font (size 1.27 1.27)) (justify left))
     )
-    (property "Footprint" "Capacitor_SMD:C_0805_2012Metric_Pad1.18x1.45mm_HandSolder" (at 207.3402 36.83 0)
+    (property "Footprint" "Capacitor_SMD:C_0603_1608Metric_Pad1.08x0.95mm_HandSolder" (at 207.3402 36.83 0)
       (effects (font (size 1.27 1.27)) hide)
     )
@@
       (effects (font (size 1.27 1.27)) (justify right))
     )
-    (property "Footprint" "Capacitor_SMD:C_0805_2012Metric_Pad1.18x1.45mm_HandSolder" (at 249.8598 37.465 0)
+    (property "Footprint" "Capacitor_SMD:C_0603_1608Metric_Pad1.08x0.95mm_HandSolder" (at 249.8598 37.465 0)
       (effects (font (size 1.27 1.27)) hide)
     )
@@
       (effects (font (size 1.27 1.27)) (justify left))
     )
-    (property "Footprint" "Capacitor_SMD:C_0805_2012Metric_Pad1.18x1.45mm_HandSolder" (at 198.4502 36.83 0)
+    (property "Footprint" "Capacitor_SMD:C_0603_1608Metric_Pad1.08x0.95mm_HandSolder" (at 198.4502 36.83 0)
       (effects (font (size 1.27 1.27)) hide)
     )
@@
       (effects (font (size 1.27 1.27)) (justify left))
     )
-    (property "Footprint" "Capacitor_SMD:C_0805_2012Metric_Pad1.18x1.45mm_HandSolder" (at 195.2752 111.125 0)
+    (property "Footprint" "Capacitor_SMD:C_0603_1608Metric_Pad1.08x0.95mm_HandSolder" (at 195.2752 111.125 0)
       (effects (font (size 1.27 1.27)) hide)
     )
@@
       (effects (font (size 1.27 1.27)) (justify left))
     )
-    (property "Footprint" "Capacitor_SMD:C_0805_2012Metric_Pad1.18x1.45mm_HandSolder" (at 86.0552 160.02 0)
+    (property "Footprint" "Capacitor_SMD:C_0603_1608Metric_Pad1.08x0.95mm_HandSolder" (at 86.0552 160.02 0)
       (effects (font (size 1.27 1.27)) hide)
     )
@@
       (effects (font (size 1.27 1.27)) (justify left))
     )
-    (property "Footprint" "Capacitor_SMD:C_0805_2012Metric_Pad1.18x1.45mm_HandSolder" (at 180.0352 175.895 0)
+    (property "Footprint" "Capacitor_SMD:C_0603_1608Metric_Pad1.08x0.95mm_HandSolder" (at 180.0352 175.895 0)
       (effects (font (size 1.27 1.27)) hide)
     )
@@
       (effects (font (size 1.27 1.27)) (justify left))
     )
-    (property "Footprint" "Capacitor_SMD:C_0805_2012Metric_Pad1.18x1.45mm_HandSolder" (at 189.5602 36.83 0)
+    (property "Footprint" "Capacitor_SMD:C_0603_1608Metric_Pad1.08x0.95mm_HandSolder" (at 189.5602 36.83 0)
       (effects (font (size 1.27 1.27)) hide)
     )
@@
       (effects (font (size 1.27 1.27)) (justify left))
     )
-    (property "Footprint" "Capacitor_SMD:C_0805_2012Metric_Pad1.18x1.45mm_HandSolder" (at 232.7402 36.83 0)
-      (effects (font (size 1.27 1.27)) hide)
-    )
+    (property "Footprint" "Capacitor_SMD:C_0603_1608Metric_Pad1.08x0.95mm_HandSolder" (at 232.7402 36.83 0)
+      (effects (font (size 1.27 1.27)) hide)
+    )

Commit message: pcb and footprints
0603
Parts:
- R10, R11, R12, R13, R14, R15, R16, R17, R18, R19, R20, R7, R8, R9: footprint Resistor_SMD:R_0805_2012Metric_Pad1.20x1.40mm_HandSolder -> Resistor_SMD:R_0603_1608Metric_Pad0.98x0.95mm_HandSolder
Changed lines of the file:
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@@
       (effects (font (size 1.27 1.27)))
     )
-    (property "Footprint" "Resistor_SMD:R_0805_2012Metric_Pad1.20x1.40mm_HandSolder" (at 307.34 144.018 90)
+    (property "Footprint" "Resistor_SMD:R_0603_1608Metric_Pad0.98x0.95mm_HandSolder" (at 307.34 144.018 90)
       (effects (font (size 1.27 1.27)) hide)
     )
@@
       (effects (font (size 1.27 1.27)))
     )
-    (property "Footprint" "Resistor_SMD:R_0805_2012Metric_Pad1.20x1.40mm_HandSolder" (at 307.34 100.838 90)
+    (property "Footprint" "Resistor_SMD:R_0603_1608Metric_Pad0.98x0.95mm_HandSolder" (at 307.34 100.838 90)
       (effects (font (size 1.27 1.27)) hide)
     )
@@
       (effects (font (size 1.27 1.27)))
     )
-    (property "Footprint" "Resistor_SMD:R_0805_2012Metric_Pad1.20x1.40mm_HandSolder" (at 307.34 131.318 90)
+    (property "Footprint" "Resistor_SMD:R_0603_1608Metric_Pad0.98x0.95mm_HandSolder" (at 307.34 131.318 90)
       (effects (font (size 1.27 1.27)) hide)
     )
@@
       (effects (font (size 1.27 1.27)))
     )
-    (property "Footprint" "Resistor_SMD:R_0805_2012Metric_Pad1.20x1.40mm_HandSolder" (at 307.34 93.218 90)
+    (property "Footprint" "Resistor_SMD:R_0603_1608Metric_Pad0.98x0.95mm_HandSolder" (at 307.34 93.218 90)
       (effects (font (size 1.27 1.27)) hide)
     )
@@
       (effects (font (size 1.27 1.27)))
     )
-    (property "Footprint" "Resistor_SMD:R_0805_2012Metric_Pad1.20x1.40mm_HandSolder" (at 307.34 128.778 90)
+    (property "Footprint" "Resistor_SMD:R_0603_1608Metric_Pad0.98x0.95mm_HandSolder" (at 307.34 128.778 90)
       (effects (font (size 1.27 1.27)) hide)
     )
@@
       (effects (font (size 1.27 1.27)))
     )
-    (property "Footprint" "Resistor_SMD:R_0805_2012Metric_Pad1.20x1.40mm_HandSolder" (at 307.34 85.598 90)
+    (property "Footprint" "Resistor_SMD:R_0603_1608Metric_Pad0.98x0.95mm_HandSolder" (at 307.34 85.598 90)
       (effects (font (size 1.27 1.27)) hide)
     )
@@
       (effects (font (size 1.27 1.27)))
     )
-    (property "Footprint" "Resistor_SMD:R_0805_2012Metric_Pad1.20x1.40mm_HandSolder" (at 307.34 88.138 90)
+    (property "Footprint" "Resistor_SMD:R_0603_1608Metric_Pad0.98x0.95mm_HandSolder" (at 307.34 88.138 90)
       (effects (font (size 1.27 1.27)) hide)
     )
@@
       (effects (font (size 1.27 1.27)))
     )
-    (property "Footprint" "Resistor_SMD:R_0805_2012Metric_Pad1.20x1.40mm_HandSolder" (at 307.34 83.058 90)
+    (property "Footprint" "Resistor_SMD:R_0603_1608Metric_Pad0.98x0.95mm_HandSolder" (at 307.34 83.058 90)
       (effects (font (size 1.27 1.27)) hide)
     )
@@
       (effects (font (size 1.27 1.27)))
     )
-    (property "Footprint" "Resistor_SMD:R_0805_2012Metric_Pad1.20x1.40mm_HandSolder" (at 307.34 138.938 90)
+    (property "Footprint" "Resistor_SMD:R_0603_1608Metric_Pad0.98x0.95mm_HandSolder" (at 307.34 138.938 90)
       (effects (font (size 1.27 1.27)) hide)
     )
@@
       (effects (font (size 1.27 1.27)))
     )
-    (property "Footprint" "Resistor_SMD:R_0805_2012Metric_Pad1.20x1.40mm_HandSolder" (at 184.785 193.548 90)
+    (property "Footprint" "Resistor_SMD:R_0603_1608Metric_Pad0.98x0.95mm_HandSolder" (at 184.785 193.548 90)
       (effects (font (size 1.27 1.27)) hide)
     )
@@
       (effects (font (size 1.27 1.27)))
     )
-    (property "Footprint" "Resistor_SMD:R_0805_2012Metric_Pad1.20x1.40mm_HandSolder" (at 307.34 141.478 90)
+    (property "Footprint" "Resistor_SMD:R_0603_1608Metric_Pad0.98x0.95mm_HandSolder" (at 307.34 141.478 90)
       (effects (font (size 1.27 1.27)) hide)
     )
@@
       (effects (font (size 1.27 1.27)))
     )
-    (property "Footprint" "Resistor_SMD:R_0805_2012Metric_Pad1.20x1.40mm_HandSolder" (at 307.34 98.298 90)
+    (property "Footprint" "Resistor_SMD:R_0603_1608Metric_Pad0.98x0.95mm_HandSolder" (at 307.34 98.298 90)
       (effects (font (size 1.27 1.27)) hide)
     )
@@
       (effects (font (size 1.27 1.27)))
     )
-    (property "Footprint" "Resistor_SMD:R_0805_2012Metric_Pad1.20x1.40mm_HandSolder" (at 307.34 133.858 90)
+    (property "Footprint" "Resistor_SMD:R_0603_1608Metric_Pad0.98x0.95mm_HandSolder" (at 307.34 133.858 90)
       (effects (font (size 1.27 1.27)) hide)
     )
@@
       (effects (font (size 1.27 1.27)))
     )
-    (property "Footprint" "Resistor_SMD:R_0805_2012Metric_Pad1.20x1.40mm_HandSolder" (at 307.34 136.398 90)
-      (effects (font (size 1.27 1.27)) hide)
-    )
+    (property "Footprint" "Resistor_SMD:R_0603_1608Metric_Pad0.98x0.95mm_HandSolder" (at 307.34 136.398 90)
+      (effects (font (size 1.27 1.27)) hide)
+    )

Commit message: pcb
added John zendong
Parts:
- added D2: GREEN, LED_SMD:LED_0805_2012Metric_Pad1.15x1.40mm_HandSolder, symbol Device:LED
- added R27: 10K, Resistor_SMD:R_0603_1608Metric_Pad0.98x0.95mm_HandSolder, symbol Device:R
- added R28: 690R, Resistor_SMD:R_0805_2012Metric_Pad1.20x1.40mm_HandSolder, symbol Device:R
- added TP7: TestPoint, TestPoint:TestPoint_Pad_1.5x1.5mm, symbol Connector:TestPoint
Connections:
- net +3V3: now also R27.1, R28.1
- net GND: now also D2.1 (K)
- net ICE_CDONE: now also D2.2 (A), R28.2
- net ICE_CREST: now also R27.2, TP7.1
