File: UFO-FPGA/Programmer.kicad_sch (KiCad schematic)
At the start: 42 parts, among them U2 FT2232HL, U3 ASDMB-12MHz, U5 93LC56CT-I/MS

Commit message: pcb
Parts:
- TP7: footprint TestPoint:TestPoint_Pad_1.5x1.5mm -> TestPoint:TestPoint_Pad_1.0x1.0mm
Connections:
- net CTSn: no longer R17.1, U2.41 (BDBUS3)
- net DCDn: no longer R20.1, U2.45 (BDBUS6)
- net DSRn: no longer R19.1, U2.44 (BDBUS5)
- net DTRn: no longer R18.2, U2.43 (BDBUS4)
- net RTSn: no longer R16.1, U2.40 (BDBUS2)
- new net CTSn-ft: R17.1, U2.41 (BDBUS3)
- new net DCDn-ft: R20.1, U2.45 (BDBUS6)
- new net DSRn-ft: R19.1, U2.44 (BDBUS5)
- new net DTRn-ft: R18.2, U2.43 (BDBUS4)
- new net RTSn-ft: R16.1, U2.40 (BDBUS2)
Other:
- moved on the sheet: R16, R17, R19, R20
Changed lines of the file:
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@@
     (effects (font (size 1.27 1.27)) (justify left bottom))
   )
-  (label "DSRn" (at 287.655 139.7 0) (fields_autoplaced)
+  (label "DSRn-ft" (at 287.655 139.7 0) (fields_autoplaced)
     (effects (font (size 1.27 1.27)) (justify left bottom))
   )
@@
     (effects (font (size 1.27 1.27)) (justify left bottom))
   )
-  (label "DTRn" (at 287.655 137.16 0) (fields_autoplaced)
+  (label "DTRn-ft" (at 287.655 137.16 0) (fields_autoplaced)
     (effects (font (size 1.27 1.27)) (justify left bottom))
   )
@@
     (effects (font (size 1.27 1.27)) (justify left bottom))
   )
-  (label "DCDn" (at 287.655 142.24 0) (fields_autoplaced)
+  (label "DCDn-ft" (at 287.655 142.24 0) (fields_autoplaced)
     (effects (font (size 1.27 1.27)) (justify left bottom))
   )
@@
     (effects (font (size 1.27 1.27)) (justify left bottom))
   )
-  (label "RTSn" (at 287.655 132.08 0) (fields_autoplaced)
+  (label "RTSn-ft" (at 287.655 132.08 0) (fields_autoplaced)
     (effects (font (size 1.27 1.27)) (justify left bottom))
   )
@@
     (effects (font (size 1.27 1.27)) (justify left bottom))
   )
-  (label "CTSn" (at 287.655 134.62 0) (fields_autoplaced)
+  (label "CTSn-ft" (at 287.655 134.62 0) (fields_autoplaced)
     (effects (font (size 1.27 1.27)) (justify left bottom))
   )
@@
     )
   )
-  (symbol (lib_id "Device:R") (at 307.34 142.24 270) (mirror x) (unit 1)
+  (symbol (lib_id "Device:R") (at 307.34 142.24 90) (mirror x) (unit 1)
     (in_bom yes) (on_board yes) (dnp no)
     (property "Reference" "R20" (at 313.055 142.24 90)
@@
       (effects (font (size 1.27 1.27)))
     )
-    (property "Footprint" "Resistor_SMD:R_0603_1608Metric_Pad0.98x0.95mm_HandSolder" (at 307.34 144.018 90)
+    (property "Footprint" "Resistor_SMD:R_0603_1608Metric_Pad0.98x0.95mm_HandSolder" (at 307.34 140.462 90)
       (effects (font (size 1.27 1.27)) hide)
     )
@@
     )
   )
-  (symbol (lib_id "Device:R") (at 307.34 139.7 270) (mirror x) (unit 1)
+  (symbol (lib_id "Device:R") (at 307.34 139.7 90) (mirror x) (unit 1)
     (in_bom yes) (on_board yes) (dnp no)
     (property "Reference" "R19" (at 313.055 139.7 90)
@@
       (effects (font (size 1.27 1.27)))
     )
-    (property "Footprint" "Resistor_SMD:R_0603_1608Metric_Pad0.98x0.95mm_HandSolder" (at 307.34 141.478 90)
+    (property "Footprint" "Resistor_SMD:R_0603_1608Metric_Pad0.98x0.95mm_HandSolder" (at 307.34 137.922 90)
       (effects (font (size 1.27 1.27)) hide)
     )
@@
     )
   )
-  (symbol (lib_id "Device:R") (at 307.34 132.08 270) (mirror x) (unit 1)
+  (symbol (lib_id "Device:R") (at 307.34 132.08 90) (mirror x) (unit 1)
     (in_bom yes) (on_board yes) (dnp no)
     (property "Reference" "R16" (at 313.055 132.08 90)
@@
       (effects (font (size 1.27 1.27)))
     )
-    (property "Footprint" "Resistor_SMD:R_0603_1608Metric_Pad0.98x0.95mm_HandSolder" (at 307.34 133.858 90)
+    (property "Footprint" "Resistor_SMD:R_0603_1608Metric_Pad0.98x0.95mm_HandSolder" (at 307.34 130.302 90)
       (effects (font (size 1.27 1.27)) hide)
     )
@@
     )
   )
-  (symbol (lib_id "Device:R") (at 307.34 134.62 270) (mirror x) (unit 1)
+  (symbol (lib_id "Device:R") (at 307.34 134.62 90) (mirror x) (unit 1)
     (in_bom yes) (on_board yes) (dnp no)
     (property "Reference" "R17" (at 313.055 134.62 90)
@@
       (effects (font (size 1.27 1.27)))
     )
-    (property "Footprint" "Resistor_SMD:R_0603_1608Metric_Pad0.98x0.95mm_HandSolder" (at 307.34 136.398 90)
+    (property "Footprint" "Resistor_SMD:R_0603_1608Metric_Pad0.98x0.95mm_HandSolder" (at 307.34 132.842 90)
       (effects (font (size 1.27 1.27)) hide)
     )
@@
       (effects (font (size 1.27 1.27)) (justify right))
     )
-    (property "Footprint" "TestPoint:TestPoint_Pad_1.5x1.5mm" (at 337.185 99.06 0)
-      (effects (font (size 1.27 1.27)) hide)
-    )
+    (property "Footprint" "TestPoint:TestPoint_Pad_1.0x1.0mm" (at 337.185 99.06 0)
+      (effects (font (size 1.27 1.27)) hide)
+    )

Commit message: pcb
Parts:
- U3: footprint Oscillator:Oscillator_SMD_Abracon_ASDMB-4Pin_2.5x2.0mm -> UFO-Footpints:ASDDV-12.000MHz-LC-T3
Changed lines of the file:
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@@
       (effects (font (size 1.27 1.27)))
     )
-    (property "Footprint" "Oscillator:Oscillator_SMD_Abracon_ASDMB-4Pin_2.5x2.0mm" (at 164.465 185.42 0)
+    (property "Footprint" "UFO-Footpints:ASDDV-12.000MHz-LC-T3" (at 164.465 185.42 0)
       (effects (font (size 1.27 1.27)) hide)
     )

Commit message: schema
Other:
- title: (none) -> FT2232H usb prog
- moved on the sheet: C1, C10, C11, C12, C13, C2, C3, C4, C7, C8, C9, D2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
