File: UFO-FPGA/BANK3.kicad_sch (KiCad schematic)
At the start: 7 parts, among them U1 ICE40HX8K-BG121

Commit message: PCB
Parts:
- TP8: footprint TestPoint:TestPoint_Keystone_5000-5004_Miniature -> TestPoint:TestPoint_Pad_1.5x1.5mm
Connections:
- net ICE_CLK: no longer U1.G1 (IOL_14A_GBIN6)
- net PIN-8: no longer U1.B2 (IOL_2B)
- net PIN-9: no longer U1.B1 (IOL_2A)
- net RS232_Tx_TTL: no longer U1.K1 (IOL_23B)
- net +1V2 renamed +3V3
- no-connect marks 0 -> 22
Changed lines of the file:
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@@
   (junction (at 174.625 37.465) (diameter 0) (color 0 0 0 0)
   )
+  (no_connect (at 117.475 94.615))
+  (no_connect (at 117.475 76.835))
+  (no_connect (at 117.475 114.935))
+  (no_connect (at 117.475 99.695))
+  (no_connect (at 117.475 89.535))
+  (no_connect (at 117.475 112.395))
+  (no_connect (at 117.475 92.075))
+  (no_connect (at 117.475 107.315))
+  (no_connect (at 117.475 122.555))
+  (no_connect (at 117.475 109.855))
+  (no_connect (at 117.475 86.995))
+  (no_connect (at 117.475 69.215))
+  (no_connect (at 117.475 71.755))
+  (no_connect (at 117.475 104.775))
+  (no_connect (at 117.475 117.475))
+  (no_connect (at 117.475 66.675))
+  (no_connect (at 117.475 125.095))
+  (no_connect (at 117.475 84.455))
+  (no_connect (at 117.475 79.375))
+  (no_connect (at 117.475 74.295))
+  (no_connect (at 117.475 81.915))
+  (no_connect (at 117.475 97.155))
   (wire (pts (xy 100.33 61.595) (xy 117.475 61.595))
     (stroke (width 0) (type default))
@@
     (effects (font (size 1.27 1.27)) (justify left bottom))
   )
-  (global_label "PIN-8" (shape input) (at 100.33 64.135 180) (fields_autoplaced)
+  (global_label "PIN-8" (shape input) (at 87.63 64.135 180) (fields_autoplaced)
     (effects (font (size 1.27 1.27)) (justify right))
-    (property "Intersheetrefs" "${INTERSHEET_REFS}" (at 91.437 64.135 0)
+    (property "Intersheetrefs" "${INTERSHEET_REFS}" (at 78.737 64.135 0)
       (effects (font (size 1.27 1.27)) (justify right) hide)
     )
   )
-  (global_label "RS232_Tx_TTL" (shape input) (at 100.33 120.015 180) (fields_autoplaced)
+  (global_label "RS232_Tx_TTL" (shape input) (at 87.63 120.015 180) (fields_autoplaced)
     (effects (font (size 1.27 1.27)) (justify right))
-    (property "Intersheetrefs" "${INTERSHEET_REFS}" (at 84.422 120.015 0)
+    (property "Intersheetrefs" "${INTERSHEET_REFS}" (at 71.722 120.015 0)
       (effects (font (size 1.27 1.27)) (justify right) hide)
     )
   )
-  (global_label "ICE_CLK" (shape input) (at 100.33 102.235 180) (fields_autoplaced)
+  (global_label "ICE_CLK" (shape input) (at 87.63 102.235 180) (fields_autoplaced)
     (effects (font (size 1.27 1.27)) (justify right))
-    (property "Intersheetrefs" "${INTERSHEET_REFS}" (at 89.8647 102.235 0)
+    (property "Intersheetrefs" "${INTERSHEET_REFS}" (at 77.1647 102.235 0)
       (effects (font (size 1.27 1.27)) (justify right) hide)
     )
   )
-  (global_label "PIN-9" (shape input) (at 100.33 61.595 180) (fields_autoplaced)
+  (global_label "PIN-9" (shape input) (at 87.63 61.595 180) (fields_autoplaced)
     (effects (font (size 1.27 1.27)) (justify right))
-    (property "Intersheetrefs" "${INTERSHEET_REFS}" (at 91.437 61.595 0)
+    (property "Intersheetrefs" "${INTERSHEET_REFS}" (at 78.737 61.595 0)
       (effects (font (size 1.27 1.27)) (justify right) hide)
     )
@@
     )
   )
-  (symbol (lib_id "power:+1V2") (at 193.675 27.305 0) (unit 1)
-    (in_bom yes) (on_board yes) (dnp no) (fields_autoplaced)
-    (property "Reference" "#PWR024" (at 193.675 31.115 0)
-      (effects (font (size 1.27 1.27)) hide)
-    )
-    (property "Value" "+1V2" (at 193.675 23.8031 0)
+  (symbol (lib_id "power:+3V3") (at 193.675 27.305 0) (unit 1)
+    (in_bom yes) (on_board yes) (dnp no) (fields_autoplaced)
+    (property "Reference" "#PWR062" (at 193.675 31.115 0)
+      (effects (font (size 1.27 1.27)) hide)
+    )
+    (property "Value" "+3V3" (at 193.675 23.8031 0)
       (effects (font (size 1.27 1.27)))
     )
@@
     (instances
       (project "UFO-FPGA"
-        (path "/b3168f6a-c732-41d3-aeeb-d97dd2f1bb65/a9a0295d-b075-4952-a5ba-04debc5f691c"
-          (reference "#PWR024") (unit 1)
-        )
         (path "/b3168f6a-c732-41d3-aeeb-d97dd2f1bb65/03eb349d-f783-448d-a9ad-735fd21dbf61"
-          (reference "#PWR027") (unit 1)
-        )
-        (path "/b3168f6a-c732-41d3-aeeb-d97dd2f1bb65/6f7e0d88-d92b-4c4f-9dc8-64721cd46d41"
-          (reference "#PWR029") (unit 1)
-        )
-        (path "/b3168f6a-c732-41d3-aeeb-d97dd2f1bb65/f54d4357-d916-4d6b-afb9-9dd5f65d1cf7"
-          (reference "#PWR036") (unit 1)
-        )
-        (path "/b3168f6a-c732-41d3-aeeb-d97dd2f1bb65/baabafd2-c41f-4db4-a640-329e074df703"
-          (reference "#PWR079") (unit 1)
-        )
-      )
-      (project "BANK3"
-        (path "/de984c47-a4b3-4404-8f6d-5958f9d846d6"
-          (reference "#PWR024") (unit 1)
+          (reference "#PWR062") (unit 1)
+        )
+        (path "/b3168f6a-c732-41d3-aeeb-d97dd2f1bb65/baabafd2-c41f-4db4-a640-329e074df703"
+          (reference "#PWR077") (unit 1)
         )
       )
@@
       (effects (font (size 1.27 1.27)) (justify left))
     )
-    (property "Footprint" "TestPoint:TestPoint_Keystone_5000-5004_Miniature" (at 180.975 37.465 0)
-      (effects (font (size 1.27 1.27)) hide)
-    )
+    (property "Footprint" "TestPoint:TestPoint_Pad_1.5x1.5mm" (at 180.975 37.465 0)
+      (effects (font (size 1.27 1.27)) hide)
+    )

Commit message: PCB
many pcb changes
-started routing
-added vias
-power planes
-ground planes
Parts:
- removed C17 (x3): 100nF, Capacitor_SMD:C_0805_2012Metric_Pad1.18x1.45mm_HandSolder, symbol Device:C
- removed R25: 1, Resistor_SMD:R_0805_2012Metric_Pad1.20x1.40mm_HandSolder, symbol Device:R
- added C17: 200nF, Capacitor_SMD:C_0805_2012Metric_Pad1.18x1.45mm_HandSolder, symbol Device:C
- added R29: 0, Resistor_SMD:R_0805_2012Metric_Pad1.20x1.40mm_HandSolder, symbol Device:R
- C18: value 100nF -> 200nF
Connections:
- net +3V3: now also R29.2
- net GND: now also C17.2
- net VCCIO_3: now also C17.1, R29.1

Commit message: pcb prog redesign
Changed lines of the file:
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@@
-    )
-  )
-  (global_label "ICE_CLK" (shape input) (at 87.63 102.235 180) (fields_autoplaced)
-    (effects (font (size 1.27 1.27)) (justify right))
-    (property "Intersheetrefs" "${INTERSHEET_REFS}" (at 77.1647 102.235 0)
-      (effects (font (size 1.27 1.27)) (justify right) hide)
     )
   )

Commit message: pcb placement
Parts:
- removed R29: 0, Resistor_SMD:R_0805_2012Metric_Pad1.20x1.40mm_HandSolder, symbol Device:R
- removed TP8: TestPoint, TestPoint:TestPoint_Pad_1.5x1.5mm, symbol Connector:TestPoint
Connections:
- net VCCIO_3 is gone; now on net +3V3: C17.1, C18.1, U1.E4 (VCCIO_3), U1.G4 (VCCIO_3)
Changed lines of the file:
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@@
     (company "Universal-Field-Objects")
-  )
-  (junction (at 175.895 37.465) (diameter 0) (color 0 0 0 0)
   )
   (junction (at 165.1 37.465) (diameter 0) (color 0 0 0 0)
@@
     (stroke (width 0) (type default))
   )
-  (wire (pts (xy 189.865 37.465) (xy 193.675 37.465))
-    (stroke (width 0) (type default))
-  )
   (wire (pts (xy 100.33 120.015) (xy 117.475 120.015))
     (stroke (width 0) (type default))
@@
     (stroke (width 0) (type default))
   )
-  (wire (pts (xy 175.895 37.465) (xy 182.245 37.465))
-    (stroke (width 0) (type default))
-  )
   (wire (pts (xy 130.175 37.465) (xy 130.175 46.355))
     (stroke (width 0) (type default))
   )
-  (wire (pts (xy 165.1 37.465) (xy 175.895 37.465))
+  (wire (pts (xy 165.1 37.465) (xy 193.675 37.465))
     (stroke (width 0) (type default))
   )
@@
     )
   )
-  (symbol (lib_id "Device:R") (at 186.055 37.465 90) (unit 1)
-    (in_bom yes) (on_board yes) (dnp no) (fields_autoplaced)
-    (property "Reference" "R29" (at 186.055 33.4391 90)
-      (effects (font (size 1.27 1.27)))
-    )
-    (property "Value" "0" (at 186.055 35.3601 90)
-      (effects (font (size 1.27 1.27)))
-    )
-    (property "Footprint" "Resistor_SMD:R_0805_2012Metric_Pad1.20x1.40mm_HandSolder" (at 186.055 39.243 90)
-      (effects (font (size 1.27 1.27)) hide)
-    )
-    (property "Datasheet" "~" (at 186.055 37.465 0)
-      (effects (font (size 1.27 1.27)) hide)
-    )
-    (pin "1")
-    (pin "2")
-    (instances
-      (project "UFO-FPGA"
-        (path "/b3168f6a-c732-41d3-aeeb-d97dd2f1bb65/f54d4357-d916-4d6b-afb9-9dd5f65d1cf7"
-          (reference "R29") (unit 1)
-        )
-        (path "/b3168f6a-c732-41d3-aeeb-d97dd2f1bb65/baabafd2-c41f-4db4-a640-329e074df703"
-          (reference "R31") (unit 1)
-        )
-      )
-    )
-  )
   (symbol (lib_id "power:GND") (at 165.1 45.085 0) (unit 1)
     (in_bom yes) (on_board yes) (dnp no) (fields_autoplaced)
@@
         )
       )
-    )
-  )
-  (symbol (lib_id "Connector:TestPoint") (at 175.895 37.465 0) (unit 1)
-    (in_bom yes) (on_board yes) (dnp no)
-    (property "Reference" "TP8" (at 174.625 30.48 0)
-      (effects (font (size 1.27 1.27)) (justify left))
-    )
-    (property "Value" "TestPoint" (at 172.085 32.385 0)
-      (effects (font (size 1.27 1.27)) (justify left))
-    )
-    (property "Footprint" "TestPoint:TestPoint_Pad_1.5x1.5mm" (at 180.975 37.465 0)
-      (effects (font (size 1.27 1.27)) hide)
-    )
-    (property "Datasheet" "~" (at 180.975 37.465 0)
-      (effects (font (size 1.27 1.27)) hide)
-    )
-    (pin "1")
-    (instances
-      (project "UFO-FPGA"
-        (path "/b3168f6a-c732-41d3-aeeb-d97dd2f1bb65/6f7e0d88-d92b-4c4f-9dc8-64721cd46d41"
-          (reference "TP8") (unit 1)
-        )
-        (path "/b3168f6a-c732-41d3-aeeb-d97dd2f1bb65/a9a0295d-b075-4952-a5ba-04debc5f691c"
-          (reference "TP5") (unit 1)
-        )
-        (path "/b3168f6a-c732-41d3-aeeb-d97dd2f1bb65/f54d4357-d916-4d6b-afb9-9dd5f65d1cf7"
-          (reference "TP9") (unit 1)
-        )
-        (path "/b3168f6a-c732-41d3-aeeb-d97dd2f1bb65/baabafd2-c41f-4db4-a640-329e074df703"
-          (reference "TP11") (unit 1)
-        )
-      )
-      (project "BANK3"
-        (path "/de984c47-a4b3-4404-8f6d-5958f9d846d6"
-          (reference "TP8") (unit 1)
-        )
-      )

Commit message: pcb 0603
Parts:
- C17, C18: footprint Capacitor_SMD:C_0805_2012Metric_Pad1.18x1.45mm_HandSolder -> Capacitor_SMD:C_0603_1608Metric_Pad1.08x0.95mm_HandSolder
Changed lines of the file:
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@@
       (effects (font (size 1.27 1.27)) (justify left))
     )
-    (property "Footprint" "Capacitor_SMD:C_0805_2012Metric_Pad1.18x1.45mm_HandSolder" (at 164.1348 45.085 0)
+    (property "Footprint" "Capacitor_SMD:C_0603_1608Metric_Pad1.08x0.95mm_HandSolder" (at 164.1348 45.085 0)
       (effects (font (size 1.27 1.27)) hide)
     )
@@
       (effects (font (size 1.27 1.27)) (justify left))
     )
-    (property "Footprint" "Capacitor_SMD:C_0805_2012Metric_Pad1.18x1.45mm_HandSolder" (at 152.7048 45.085 0)
+    (property "Footprint" "Capacitor_SMD:C_0603_1608Metric_Pad1.08x0.95mm_HandSolder" (at 152.7048 45.085 0)
       (effects (font (size 1.27 1.27)) hide)
     )

Commit message: pcb
added John zendong
Parts:
- removed U1: ICE40HX8K-BG121, Package_BGA:BGA-121_9.0x9.0mm_Layout11x11_P0.8mm_Ball0.4mm_Pad0.35mm_NSMD, symbol FPGA_Lattice:ICE40HX8K-BG121
- added U4: ICE40HX4K-TQ144, Package_QFP:TQFP-144_20x20mm_P0.5mm, symbol FPGA_Lattice:ICE40HX4K-TQ144
Connections:
- net +3V3: now also U4.30 (VCCIO_3), U4.6 (VCCIO_3)

Commit message: pcb
Connections:
- net DCDn: now reaches U4.31 (IOL_24A)
- net DSRn: now reaches U4.32 (IOL_24B)
- net DTRn: now reaches U4.33 (IOL_25A)
- net CTSn: now reaches U4.34 (IOL_25B)
- no-connect marks 22 -> 19
Changed lines of the file:
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@@
   (junction (at 153.67 37.465) (diameter 0) (color 0 0 0 0)
   )
+  (no_connect (at 117.475 102.235))
   (no_connect (at 117.475 94.615))
   (no_connect (at 117.475 76.835))
@@
   (no_connect (at 117.475 112.395))
   (no_connect (at 117.475 92.075))
-  (no_connect (at 117.475 107.315))
-  (no_connect (at 117.475 122.555))
-  (no_connect (at 117.475 109.855))
   (no_connect (at 117.475 86.995))
   (no_connect (at 117.475 69.215))
   (no_connect (at 117.475 71.755))
-  (no_connect (at 117.475 104.775))
+  (no_connect (at 117.475 120.015))
   (no_connect (at 117.475 117.475))
   (no_connect (at 117.475 66.675))
-  (no_connect (at 117.475 125.095))
   (no_connect (at 117.475 84.455))
   (no_connect (at 117.475 79.375))
@@
     (stroke (width 0) (type default))
   )
-  (wire (pts (xy 100.33 120.015) (xy 117.475 120.015))
+  (wire (pts (xy 100.33 109.855) (xy 117.475 109.855))
+    (stroke (width 0) (type default))
+  )
+  (wire (pts (xy 100.33 125.095) (xy 117.475 125.095))
     (stroke (width 0) (type default))
   )
@@
     (stroke (width 0) (type default))
   )
-  (wire (pts (xy 100.33 102.235) (xy 117.475 102.235))
+  (wire (pts (xy 100.33 130.175) (xy 117.475 130.175))
     (stroke (width 0) (type default))
   )
   (wire (pts (xy 130.175 37.465) (xy 153.67 37.465))
+    (stroke (width 0) (type default))
+  )
+  (wire (pts (xy 100.33 127.635) (xy 117.475 127.635))
+    (stroke (width 0) (type default))
+  )
+  (wire (pts (xy 100.33 104.775) (xy 117.475 104.775))
+    (stroke (width 0) (type default))
+  )
+  (wire (pts (xy 100.33 107.315) (xy 117.475 107.315))
     (stroke (width 0) (type default))
   )
@@
   )
   (wire (pts (xy 165.1 37.465) (xy 193.675 37.465))
+    (stroke (width 0) (type default))
+  )
+  (wire (pts (xy 100.33 122.555) (xy 117.475 122.555))
     (stroke (width 0) (type default))
   )
@@
     (effects (font (size 1.27 1.27)) (justify left bottom))
   )
+  (global_label "DTRn" (shape input) (at 100.33 127.635 180) (fields_autoplaced)
+    (effects (font (size 1.27 1.27)) (justify right))
+    (property "Intersheetrefs" "${INTERSHEET_REFS}" (at 92.7676 127.635 0)
+      (effects (font (size 1.27 1.27)) (justify right) hide)
+    )
+  )
   (global_label "PIN-8" (shape input) (at 87.63 64.135 180) (fields_autoplaced)
     (effects (font (size 1.27 1.27)) (justify right))
@@
     )
   )
-  (global_label "RS232_Tx_TTL" (shape input) (at 87.63 120.015 180) (fields_autoplaced)
+  (global_label "DCDn" (shape input) (at 100.33 122.555 180) (fields_autoplaced)
     (effects (font (size 1.27 1.27)) (justify right))
-    (property "Intersheetrefs" "${INTERSHEET_REFS}" (at 71.722 120.015 0)
+    (property "Intersheetrefs" "${INTERSHEET_REFS}" (at 92.4652 122.555 0)
       (effects (font (size 1.27 1.27)) (justify right) hide)
     )
@@
       (effects (font (size 1.27 1.27)) (justify right) hide)
     )
+  )
+  (global_label "CTSn" (shape input) (at 100.33 130.175 180) (fields_autoplaced)
+    (effects (font (size 1.27 1.27)) (justify right))
+    (property "Intersheetrefs" "${INTERSHEET_REFS}" (at 92.8281 130.175 0)
+      (effects (font (size 1.27 1.27)) (justify right) hide)
+    )
+  )
+  (global_label "DSRn" (shape input) (at 100.33 125.095 180) (fields_autoplaced)
+    (effects (font (size 1.27 1.27)) (justify right))
+    (property "Intersheetrefs" "${INTERSHEET_REFS}" (at 92.5257 125.095 0)
+      (effects (font (size 1.27 1.27)) (justify right) hide)
+    )
