File: UFO-FPGA/BANK3.kicad_sch (KiCad schematic)
At the start: 3 parts, among them U4 ICE40HX4K-TQ144

Commit message: pcb
added monkey
Connections:
- net PIN-8: now also U4.16 (IOL_10B)
- net PIN-9: now also U4.15 (IOL_10A)
- net PIN-12: now reaches U4.10 (IOL_5B)
- net PIN-11: now reaches U4.11 (IOL_8A)
- net PIN-10: now reaches U4.12 (IOL_8B)
- net PIN-7: now reaches U4.17 (IOL_12A)
- net PIN-6: now reaches U4.18 (IOL_12B)
- net PIN-5: now reaches U4.19 (IOL_13A)
- net PIN-4: now reaches U4.20 (IOL_13B_GBIN7)
- net PIN-3: now reaches U4.21 (IOL_14A_GBIN6)
- net PIN-2: now reaches U4.22 (IOL_14B)
- net PIN-1: now reaches U4.23 (IOL_17A)
- net PIN-17: now reaches U4.3 (IOL_3A)
- net PIN-16: now reaches U4.4 (IOL_3B)
- net PIN-15: now reaches U4.7 (IOL_4A)
- net PIN-14: now reaches U4.8 (IOL_4B)
- net PIN-13: now reaches U4.9 (IOL_5A)
- no-connect marks 19 -> 5
Changed lines of the file:
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@@
   (junction (at 153.67 37.465) (diameter 0) (color 0 0 0 0)
   )
-  (no_connect (at 117.475 102.235))
-  (no_connect (at 117.475 94.615))
-  (no_connect (at 117.475 76.835))
   (no_connect (at 117.475 114.935))
-  (no_connect (at 117.475 99.695))
-  (no_connect (at 117.475 89.535))
-  (no_connect (at 117.475 112.395))
-  (no_connect (at 117.475 92.075))
-  (no_connect (at 117.475 86.995))
-  (no_connect (at 117.475 69.215))
-  (no_connect (at 117.475 71.755))
   (no_connect (at 117.475 120.015))
   (no_connect (at 117.475 117.475))
-  (no_connect (at 117.475 66.675))
-  (no_connect (at 117.475 84.455))
-  (no_connect (at 117.475 79.375))
-  (no_connect (at 117.475 74.295))
-  (no_connect (at 117.475 81.915))
-  (no_connect (at 117.475 97.155))
+  (no_connect (at 117.475 64.135))
+  (no_connect (at 117.475 61.595))
   (wire (pts (xy 153.67 37.465) (xy 165.1 37.465))
     (stroke (width 0) (type default))
   )
-  (wire (pts (xy 100.33 61.595) (xy 117.475 61.595))
-    (stroke (width 0) (type default))
-  )
-  (wire (pts (xy 100.33 109.855) (xy 117.475 109.855))
+  (wire (pts (xy 100.33 107.315) (xy 117.475 107.315))
+    (stroke (width 0) (type default))
+  )
+  (wire (pts (xy 100.33 69.215) (xy 117.475 69.215))
+    (stroke (width 0) (type default))
+  )
+  (wire (pts (xy 100.33 104.775) (xy 117.475 104.775))
+    (stroke (width 0) (type default))
+  )
+  (wire (pts (xy 100.33 71.755) (xy 117.475 71.755))
+    (stroke (width 0) (type default))
+  )
+  (wire (pts (xy 100.33 76.835) (xy 117.475 76.835))
+    (stroke (width 0) (type default))
+  )
+  (wire (pts (xy 100.33 89.535) (xy 117.475 89.535))
+    (stroke (width 0) (type default))
+  )
+  (wire (pts (xy 100.33 79.375) (xy 117.475 79.375))
+    (stroke (width 0) (type default))
+  )
+  (wire (pts (xy 100.33 97.155) (xy 117.475 97.155))
+    (stroke (width 0) (type default))
+  )
+  (wire (pts (xy 100.33 66.675) (xy 117.475 66.675))
     (stroke (width 0) (type default))
   )
@@
     (stroke (width 0) (type default))
   )
+  (wire (pts (xy 100.33 92.075) (xy 117.475 92.075))
+    (stroke (width 0) (type default))
+  )
   (wire (pts (xy 153.67 45.085) (xy 165.1 45.085))
     (stroke (width 0) (type default))
   )
+  (wire (pts (xy 100.33 84.455) (xy 117.475 84.455))
+    (stroke (width 0) (type default))
+  )
   (wire (pts (xy 100.33 130.175) (xy 117.475 130.175))
     (stroke (width 0) (type default))
@@
     (stroke (width 0) (type default))
   )
-  (wire (pts (xy 100.33 104.775) (xy 117.475 104.775))
-    (stroke (width 0) (type default))
-  )
-  (wire (pts (xy 100.33 107.315) (xy 117.475 107.315))
+  (wire (pts (xy 100.33 99.695) (xy 117.475 99.695))
+    (stroke (width 0) (type default))
+  )
+  (wire (pts (xy 100.33 102.235) (xy 117.475 102.235))
     (stroke (width 0) (type default))
   )
@@
     (stroke (width 0) (type default))
   )
+  (wire (pts (xy 100.33 81.915) (xy 117.475 81.915))
+    (stroke (width 0) (type default))
+  )
   (wire (pts (xy 100.33 122.555) (xy 117.475 122.555))
     (stroke (width 0) (type default))
   )
+  (wire (pts (xy 100.33 86.995) (xy 117.475 86.995))
+    (stroke (width 0) (type default))
+  )
+  (wire (pts (xy 100.33 74.295) (xy 117.475 74.295))
+    (stroke (width 0) (type default))
+  )
+  (wire (pts (xy 100.33 94.615) (xy 117.475 94.615))
+    (stroke (width 0) (type default))
+  )
   (wire (pts (xy 193.675 27.305) (xy 193.675 37.465))
     (stroke (width 0) (type default))
   )
-  (wire (pts (xy 100.33 64.135) (xy 117.475 64.135))
-    (stroke (width 0) (type default))
-  )
-  (label "VCCIO_3" (at 130.175 37.465 0) (fields_autoplaced)
-    (effects (font (size 1.27 1.27)) (justify left bottom))
-  )
   (global_label "DTRn" (shape input) (at 100.33 127.635 180) (fields_autoplaced)
     (effects (font (size 1.27 1.27)) (justify right))
@@
     )
   )
-  (global_label "PIN-8" (shape input) (at 87.63 64.135 180) (fields_autoplaced)
-    (effects (font (size 1.27 1.27)) (justify right))
-    (property "Intersheetrefs" "${INTERSHEET_REFS}" (at 78.737 64.135 0)
+  (global_label "PIN-17" (shape input) (at 100.33 66.675 180) (fields_autoplaced)
+    (effects (font (size 1.27 1.27)) (justify right))
+    (property "Intersheetrefs" "${INTERSHEET_REFS}" (at 90.2275 66.675 0)
+      (effects (font (size 1.27 1.27)) (justify right) hide)
+    )
+  )
+  (global_label "PIN-6" (shape input) (at 100.33 94.615 180) (fields_autoplaced)
+    (effects (font (size 1.27 1.27)) (justify right))
+    (property "Intersheetrefs" "${INTERSHEET_REFS}" (at 91.437 94.615 0)
+      (effects (font (size 1.27 1.27)) (justify right) hide)
+    )
+  )
+  (global_label "PIN-2" (shape input) (at 100.33 104.775 180) (fields_autoplaced)
+    (effects (font (size 1.27 1.27)) (justify right))
+    (property "Intersheetrefs" "${INTERSHEET_REFS}" (at 91.437 104.775 0)
+      (effects (font (size 1.27 1.27)) (justify right) hide)
+    )
+  )
+  (global_label "PIN-9" (shape input) (at 100.33 86.995 180) (fields_autoplaced)
+    (effects (font (size 1.27 1.27)) (justify right))
+    (property "Intersheetrefs" "${INTERSHEET_REFS}" (at 91.437 86.995 0)
+      (effects (font (size 1.27 1.27)) (justify right) hide)
+    )
+  )
+  (global_label "PIN-13" (shape input) (at 100.33 76.835 180) (fields_autoplaced)
+    (effects (font (size 1.27 1.27)) (justify right))
+    (property "Intersheetrefs" "${INTERSHEET_REFS}" (at 90.2275 76.835 0)
+      (effects (font (size 1.27 1.27)) (justify right) hide)
+    )
+  )
+  (global_label "PIN-16" (shape input) (at 100.33 69.215 180) (fields_autoplaced)
+    (effects (font (size 1.27 1.27)) (justify right))
+    (property "Intersheetrefs" "${INTERSHEET_REFS}" (at 90.2275 69.215 0)
+      (effects (font (size 1.27 1.27)) (justify right) hide)
+    )
+  )
+  (global_label "PIN-11" (shape input) (at 100.33 81.915 180) (fields_autoplaced)
+    (effects (font (size 1.27 1.27)) (justify right))
+    (property "Intersheetrefs" "${INTERSHEET_REFS}" (at 90.2275 81.915 0)
+      (effects (font (size 1.27 1.27)) (justify right) hide)
+    )
+  )
+  (global_label "PIN-10" (shape input) (at 100.33 84.455 180) (fields_autoplaced)
+    (effects (font (size 1.27 1.27)) (justify right))
+    (property "Intersheetrefs" "${INTERSHEET_REFS}" (at 90.2275 84.455 0)
+      (effects (font (size 1.27 1.27)) (justify right) hide)
+    )
+  )
+  (global_label "PIN-8" (shape input) (at 100.33 89.535 180) (fields_autoplaced)
+    (effects (font (size 1.27 1.27)) (justify right))
+    (property "Intersheetrefs" "${INTERSHEET_REFS}" (at 91.437 89.535 0)
       (effects (font (size 1.27 1.27)) (justify right) hide)
     )
@@
     )
   )
-  (global_label "PIN-9" (shape input) (at 87.63 61.595 180) (fields_autoplaced)
-    (effects (font (size 1.27 1.27)) (justify right))
-    (property "Intersheetrefs" "${INTERSHEET_REFS}" (at 78.737 61.595 0)
+  (global_label "PIN-15" (shape input) (at 100.33 71.755 180) (fields_autoplaced)
+    (effects (font (size 1.27 1.27)) (justify right))
+    (property "Intersheetrefs" "${INTERSHEET_REFS}" (at 90.2275 71.755 0)
+      (effects (font (size 1.27 1.27)) (justify right) hide)
+    )
+  )
+  (global_label "PIN-5" (shape input) (at 100.33 97.155 180) (fields_autoplaced)
+    (effects (font (size 1.27 1.27)) (justify right))
+    (property "Intersheetrefs" "${INTERSHEET_REFS}" (at 91.437 97.155 0)
+      (effects (font (size 1.27 1.27)) (justify right) hide)
+    )
+  )
+  (global_label "PIN-14" (shape input) (at 100.33 74.295 180) (fields_autoplaced)
+    (effects (font (size 1.27 1.27)) (justify right))
+    (property "Intersheetrefs" "${INTERSHEET_REFS}" (at 90.2275 74.295 0)
+      (effects (font (size 1.27 1.27)) (justify right) hide)
+    )
+  )
+  (global_label "PIN-1" (shape input) (at 100.33 107.315 180) (fields_autoplaced)
+    (effects (font (size 1.27 1.27)) (justify right))
+    (property "Intersheetrefs" "${INTERSHEET_REFS}" (at 91.437 107.315 0)
+      (effects (font (size 1.27 1.27)) (justify right) hide)
+    )
+  )
+  (global_label "PIN-4" (shape input) (at 100.33 99.695 180) (fields_autoplaced)
+    (effects (font (size 1.27 1.27)) (justify right))
+    (property "Intersheetrefs" "${INTERSHEET_REFS}" (at 91.437 99.695 0)
+      (effects (font (size 1.27 1.27)) (justify right) hide)
+    )
+  )
+  (global_label "PIN-7" (shape input) (at 100.33 92.075 180) (fields_autoplaced)
+    (effects (font (size 1.27 1.27)) (justify right))
+    (property "Intersheetrefs" "${INTERSHEET_REFS}" (at 91.437 92.075 0)
+      (effects (font (size 1.27 1.27)) (justify right) hide)
+    )
+  )
+  (global_label "PIN-3" (shape input) (at 100.33 102.235 180) (fields_autoplaced)
+    (effects (font (size 1.27 1.27)) (justify right))
+    (property "Intersheetrefs" "${INTERSHEET_REFS}" (at 91.437 102.235 0)
       (effects (font (size 1.27 1.27)) (justify right) hide)
     )
@@
       (effects (font (size 1.27 1.27)) (justify right) hide)
     )
+  )
+  (global_label "PIN-12" (shape input) (at 100.33 79.375 180) (fields_autoplaced)
+    (effects (font (size 1.27 1.27)) (justify right))
+    (property "Intersheetrefs" "${INTERSHEET_REFS}" (at 90.2275 79.375 0)
+      (effects (font (size 1.27 1.27)) (justify right) hide)
+    )
