File: UFO-FPGA/UFO-FPGA.kicad_sch (KiCad schematic)
At the start: 0 parts

Commit message: pinout tab
Other:
- added sheet PINOUT (PINOUT.kicad_sch)
Changed lines of the file:
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@@
 (kicad_sch (version 20230121) (generator eeschema)
   (paper "A4")
+  (title_block
+    (date "2023-04-22")
+    (rev "V0.1")
+  )
   (rectangle (start 70.485 18.415) (end 158.75 66.675)
     (stroke (width 0) (type default))
@@
       (project "UFO-FPGA"
         (path "/b3168f6a-c732-41d3-aeeb-d97dd2f1bb65" (page "7"))
+      )
+    )
+  )
+  (sheet (at 161.29 21.59) (size 40.64 36.83) (fields_autoplaced)
+    (stroke (width 0.1524) (type solid))
+    (fill (color 0 0 0 0.0000))
+    (property "Sheetname" "PINOUT" (at 161.29 20.8784 0)
+      (effects (font (size 1.27 1.27)) (justify left bottom))
+    )
+    (property "Sheetfile" "PINOUT.kicad_sch" (at 161.29 59.0046 0)
+      (effects (font (size 1.27 1.27)) (justify left top) hide)
+    )
+    (instances
+      (project "UFO-FPGA"
+        (path "/b3168f6a-c732-41d3-aeeb-d97dd2f1bb65" (page "9"))
       )
     )
@@
   )
   (sheet_instances
-    (path "/" (page "5"))
+    (path "/" (page "1"))
   )
 )

Commit message: symbols
Other:
- added sheet ADC (ADC.kicad_sch)
Changed lines of the file:
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@@
+    (instances
+      (project "UFO-FPGA"
+        (path "/b3168f6a-c732-41d3-aeeb-d97dd2f1bb65" (page "10"))
+      )
+    )
+  )
+  (sheet (at 27.305 127) (size 40.64 35.56) (fields_autoplaced)
+    (stroke (width 0.1524) (type solid))
+    (fill (color 0 0 0 0.0000))
+    (property "Sheetname" "ADC" (at 27.305 126.2884 0)
+      (effects (font (size 1.27 1.27)) (justify left bottom))
+    )
+    (property "Sheetfile" "ADC.kicad_sch" (at 27.305 163.1446 0)
+      (effects (font (size 1.27 1.27)) (justify left top))
+    )
     (instances
       (project "UFO-FPGA"

Commit message: Dual ramp  MC34 inverting converter added
Other:
- added sheet Invert-5V-Dual-Ramp (untitled.kicad_sch)
Changed lines of the file:
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@@
+    )
+  )
+  (sheet (at 71.755 128.27) (size 39.37 34.29) (fields_autoplaced)
+    (stroke (width 0.1524) (type solid))
+    (fill (color 0 0 0 0.0000))
+    (property "Sheetname" "Invert-5V-Dual-Ramp" (at 71.755 127.5584 0)
+      (effects (font (size 1.27 1.27)) (justify left bottom))
+    )
+    (property "Sheetfile" "untitled.kicad_sch" (at 71.755 163.1446 0)
+      (effects (font (size 1.27 1.27)) (justify left top))
+    )
+    (instances
+      (project "UFO-FPGA"
+        (path "/b3168f6a-c732-41d3-aeeb-d97dd2f1bb65" (page "11"))
+      )
     )
   )

Commit message: IO and power
Other:
- sheet Invert-5V-Dual-Ramp: file untitled.kicad_sch -> Invert-5V-Dual-Ramp.kicad_sch
Changed lines of the file:
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@@
       (effects (font (size 1.27 1.27)) (justify left bottom))
     )
-    (property "Sheetfile" "untitled.kicad_sch" (at 71.755 163.1446 0)
+    (property "Sheetfile" "Invert-5V-Dual-Ramp.kicad_sch" (at 71.755 163.1446 0)
       (effects (font (size 1.27 1.27)) (justify left top))
     )

Commit message: Opamp gemaakt van de ADC
Enkel nog begrijpen wat VDC is. Aan docent vragen?
Other:
- sheet Invert-5V-Dual-Ramp: file Invert-5V-Dual-Ramp.kicad_sch -> untitled.kicad_sch
Changed lines of the file:
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@@
       (effects (font (size 1.27 1.27)) (justify left bottom))
     )
-    (property "Sheetfile" "Invert-5V-Dual-Ramp.kicad_sch" (at 71.755 163.1446 0)
+    (property "Sheetfile" "untitled.kicad_sch" (at 71.755 163.1446 0)
       (effects (font (size 1.27 1.27)) (justify left top))
     )

Commit message: Revision
Other:
- company: (none) -> Universal-Field-Objects
Changed lines of the file:
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@@
   (paper "A4")
   (title_block
-    (date "2023-04-22")
-    (rev "V0.1")
+    (date "2023-04-25")
+    (rev "V0.5")
+    (company "Universal-Field-Objects")
   )
   (rectangle (start 70.485 18.415) (end 158.75 66.675)

Commit message: pcb prog redesign
Other:
- removed sheet Invert-5V-Dual-Ramp
Changed lines of the file:
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@@
-    )
-  )
-  (sheet (at 71.755 128.27) (size 39.37 34.29) (fields_autoplaced)
-    (stroke (width 0.1524) (type solid))
-    (fill (color 0 0 0 0.0000))
-    (property "Sheetname" "Invert-5V-Dual-Ramp" (at 71.755 127.5584 0)
-      (effects (font (size 1.27 1.27)) (justify left bottom))
-    )
-    (property "Sheetfile" "untitled.kicad_sch" (at 71.755 163.1446 0)
-      (effects (font (size 1.27 1.27)) (justify left top))
-    )
-    (instances
-      (project "UFO-FPGA"
-        (path "/b3168f6a-c732-41d3-aeeb-d97dd2f1bb65" (page "11"))
-      )
     )
   )

Commit message: schema
Other:
- sheet BANK 4 - SPI Programming renamed SPI Programming
- note added: "+1V2"
- note added: "+3V3"
- note added: "GPIO"
- note added: "ICE40 FPGA"
- note added: "PINOUT"
- note added: "SPI"
- note added: "UART"
- title: (none) -> UFO-FPGA BLOCK diagram
